File: hw/SD-MSZ/SD-MSZ.kicad_sch (KiCad schematic)
At the start: 0 parts

Commit message: Update gitignore to skip KiCad lock and backup files.
Other:
- company: Silky Design -> SilkyDESIGN
- title: SilkyDesign MicroSystem Z80 w/Front Panel -> MicroSystem Z80 w/Front Panel & RC2014 Bus
Changed lines of the file:
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@@
 	(paper "User" 419.1 323.85)
 	(title_block
-		(title "SilkyDesign MicroSystem Z80 w/Front Panel")
-		(date "2025-08-15")
+		(title "MicroSystem Z80 w/Front Panel & RC2014 Bus")
+		(date "2025-09-22")
 		(rev "v1.0")
-		(company "Silky Design")
-		(comment 1 "Copyright AESilky 2025")
+		(company "SilkyDESIGN")
+		(comment 1 "Copyright 2025 AESilky")
+		(comment 3 "MicroSystem Z80 w/Front Panel & RC2014 Bus")
 	)
 	(sheet
