File: hw/SD-MSZ/logic_pwr_spr.kicad_sch (KiCad schematic)
At the start: 14 parts, among them U1 74HCT08, U10 74HCT11, U14 74HCT74, U23 74HCT74, U3 74HCT32, U5 74HCT14, U8 74HCT393

Commit message: Update gitignore to skip KiCad lock and backup files.
Other:
- company: Silky Design -> SilkyDESIGN
- title: Main Board - Logic Power & Spares -> Logic Power & Spares
Changed lines of the file:
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@@
 	(paper "User" 419.1 323.85)
 	(title_block
-		(title "Main Board - Logic Power & Spares")
-		(date "2025-08-15")
+		(title "Logic Power & Spares")
+		(date "2025-09-22")
 		(rev "v1.0")
-		(company "Silky Design")
-		(comment 1 "Copyright AESilky 2025")
+		(company "SilkyDESIGN")
+		(comment 1 "Copyright 2025 AESilky")
+		(comment 3 "MicroSystem Z80 w/Front Panel & RC2014 Bus")
 	)
 	(junction
