File: hw/SD-MSZ/mb_mmu.kicad_sch (KiCad schematic)
At the start: 18 parts, among them J4 Conn_02x10, U1 74HCT08, U17 74HC670, U18 74ACT244, U19 AS6C4008, U20 SST39SF040, U21 74HC670, U22 74HCT138, U23 74HCT74

Commit message: Update gitignore to skip KiCad lock and backup files.
Parts:
- U20: Part (none) -> Flash ROM
- U22: value 74HCT138 -> 74ACT138
Other:
- company: Silky Design -> SilkyDESIGN
- title: Main Board - MMU and Memory -> MMU and Memory
Changed lines of the file:
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@@
 	(paper "User" 419.1 323.85)
 	(title_block
-		(title "Main Board - MMU and Memory")
-		(date "2025-08-15")
+		(title "MMU and Memory")
+		(date "2025-09-22")
 		(rev "v1.0")
-		(company "Silky Design")
-		(comment 1 "Copyright AESilky 2025")
+		(company "SilkyDESIGN")
+		(comment 1 "Copyright 2025 AESilky")
+		(comment 3 "MicroSystem Z80 w/Front Panel & RC2014 Bus")
 	)
 	(junction
@@
 			)
 		)
-		(property "Value" "74HCT138"
+		(property "Value" "74ACT138"
 			(at 281.178 158.75 0)
 			(effects
@@
 				)
 			)
+		)
+		(property "Part" "Flash ROM"
+			(at 358.394 137.668 0)
+			(effects
+				(font
+					(size 1.27 1.27)
+					(color 0 72 72 1)
+				)
+			)
