File: hw/SD-ZMB/exp-ifc.kicad_sch (KiCad schematic)
At the start: 51 parts, among them J11 Conn_02x03, J15 Screw_Terminal_01x02, J5 Conn_02x02 HDR, J7 CONN 02x05 - DTE_HDR-AES, J8 Conn_02x05 HDR, J9 BARREL JACK

Commit message: PR7.4: checkpoint only
Parts:
- removed U?: 74HCT14, symbol AES_Library:74HC14-AES
- added U? (x3): 74HCT08, symbol 74xx:74LS08
- added U?: 74HC04, symbol AES_Library:7404-AES
- J?: Function BP80 BUS -> BP80 BUS (2)
- J?: Function BP80 BUS -> BP80 BUS (1)
Connections:
- net CTCIEO: now also U?.2; no longer U?7.6 (IEI)
- net LCD_EN: now also U?.8
- net LCD_SEL-: now also U?.9
- net SIOIEO: now also U?6.13 (IEI), U?.1
- net VPU?0: now also U?7.6 (IEI); no longer U?6.13 (IEI)
- net B2IEI: now reaches J?.80 (IEI)
- net B2IEI: now also U?.3
- net B1IEO: now reaches J?.40 (IEO)
- net B1IEO: now also U?.1
- net B1IEI: now reaches J?.80 (IEI)
- net B1IEI: now also U?.2, U?.3
- net B0IEO: now reaches J?.20 (Pin_20)
- net B0IEO: now also U?.1
- net LCLIEO: now reaches J?.40 (Pin_40)
- net LCLIEO: now also U?.2, U?.3
Other:
- moved on the sheet: J?
