File: hw/SD-ZMB/exp-ifc.kicad_sch (KiCad schematic)
At the start: 54 parts, among them J11 Conn_02x03, J15 Screw_Terminal_01x02, J5 Conn_02x02 HDR, J7 CONN 02x05 - DTE_HDR-AES, J8 Conn_02x05 HDR, J9 BARREL JACK

Commit message: ZMB: Diagrams and start of PCB. DBG: Updated WAIT. DADPT: Display/Cable PCB ordered.
Parts:
- removed C18, C19, C?: 0.1uF, symbol Device:C_Small
- removed C23: 10uF, symbol Device:C_Polarized_Small_US
- removed D3: LED RED, symbol Device:LED
- removed DS?: WC1602A, Display:WC1602A, symbol Display_Character:WC1602A
- removed J5: Conn_02x02 HDR, symbol Connector_Generic:Conn_02x02_Odd_Even
- removed J?: HDR 1x3 Pin, symbol Connector_Generic:Conn_01x03
- removed J?: SOCKET 02x40 (BRD-CONN), symbol AES_Library:RC2014_BUS_BP80-AES
- removed J?: HDR 2x3 PIN, symbol Connector_Generic:Conn_02x03_Row_Letter_First
- removed Q?: 2N3904, Package_TO_SOT_SMD:SOT-23, symbol Transistor_BJT:MMBT3904
- removed R23: 22, symbol Device:R_Small_US
- removed R24: 430, symbol Device:R_Small_US
- removed R34: 1k, symbol Device:R_Small_US
- removed R?: 15k, symbol Device:R_Small_US
- removed R?: 330, symbol AES_Library:R_PWRSRC_sm-AES
- removed RV?: 10k, symbol Device:R_Potentiometer_US
- removed U? (x3): 74HCT08, symbol 74xx:74LS08
- removed U?: 74HC04, symbol AES_Library:7404-AES
- added C4: 220uF, Capacitor_THT:CP_Radial_D6.3mm_P2.50mm, symbol Device:C_Polarized_Small_US
- added D6: CDBF0130R, Diode_SMD:D_SOD-323F, symbol AES_Library:AES-Schottky_Diode_PWR_Input
- added H8: MountingHole, MountingHole:MountingHole_3.2mm_M3, symbol Mechanical:MountingHole
- added J11, J18, J20, J7: HDR 1x02 Pin, Connector_PinHeader_2.54mm:PinHeader_1x02_P2.54mm_Vertical, symbol Connector_Generic:Conn_01x02
- added J13: HDR 02x03 PIN, AES_Library:PinHeader_2x03_AB-AES, symbol Connector_Generic:Conn_02x03_Row_Letter_First
- added J16, J21: HDR 1x3 Pin, Connector_PinHeader_2.54mm:PinHeader_1x03_P2.54mm_Vertical, symbol Connector_Generic:Conn_01x03
- added J17: HDR 2x10 Pin, Connector_PinHeader_2.54mm:PinHeader_2x10_P2.54mm_Vertical, symbol Connector_Generic:Conn_02x10_Odd_Even
- added J19: Conn_02x03, AES_Library:PinHeader_2x03_AB-AES, symbol Connector_Generic:Conn_02x03_Row_Letter_First
- added J5: HDR 02x02, AES_Library:PinHeader_2x02_AB-AES, symbol Connector_Generic:Conn_02x02_Row_Letter_First
- added Mod1: Adafruit KB2040 Module, AES_Library:Adafruit-KB2040-AES, symbol AES_Library:Adafruit-KB2040-AES
- added Q1: MMBT3904, Package_TO_SOT_SMD:SOT-23, symbol Transistor_BJT:MMBT3904
- added R19: 100, Resistor_SMD:R_0805_2012Metric_Pad1.20x1.40mm_HandSolder, symbol Device:R_Small_US
- added SD1: MicroSD-Socket, AES_Library:AES-SDCard-GCT_MEM2075-00-140-01-A, symbol Connector:Micro_SD_Card_Det1
- added SW2: SW Toggle PCB, AES_Library:SW-SPDT-PCB-TGL-RA-AES, symbol Switch:SW_SPDT
- added U11: 74AHCT74DR, Package_SO:SOIC-14_3.9x8.7mm_P1.27mm, symbol 74xx:74HC74
- added U34: 74AHCT10, Package_SO:SOIC-14_3.9x8.7mm_P1.27mm, symbol 74xx:74LS10
- added U36: SN74LVC8T245NS, Package_SO:SO-24_5.3x15mm_P1.27mm, symbol AES_Library:SN74LVC8T245-AES
- added U37: 74AHCT1G02, Package_TO_SOT_SMD:SOT-23-5, symbol AES_Library:74x1G02-AES
- added U4, U5: 74AHCT08, Package_SO:SOIC-14_3.9x8.7mm_P1.27mm, symbol 74xx:74LS08
- added U? (x5): 74LVC125, symbol 74xx:74LVC125
- C2, C5: renamed from C?; footprint (none) -> Capacitor_SMD:C_0603_1608Metric_Pad1.08x0.95mm_HandSolder
- C3: renamed from C21; value 10uF -> 220uF; footprint (none) -> Capacitor_THT:CP_Radial_D6.3mm_P2.50mm; Voltage (none) -> 25V
- C6: renamed from C?; value 100u E -> 47uF; footprint (none) -> Capacitor_THT:CP_Radial_D4.0mm_P1.50mm; Voltage (none) -> 25V
- J10: renamed from J11; footprint (none) -> AES_Library:PinHeader_2x03_AB-AES; Function CTC3 Clk Sel -> CTC3 CLK; Opt1 (none) -> 2OUT; Opt2 (none) -> CLK2; Opt3 (none) -> BCLK
- J12: renamed from J?; footprint (none) -> AES_Library:RC80-BUS-BPMB-AES; PartOpt1 (none) -> 2x 40 SIP Socket; PartOpt2 (none) -> 2x 2x20 Socket; PartOr (none) -> or
- J14: renamed from J7; footprint (none) -> AES_Library:AES-PinHeader_2x05_DB9-Order
- J15: renamed from J8; footprint (none) -> AES_Library:PinHeader_2x05_AB-AES; Function COM1_ISO -> COM1 ISO
- J3: renamed from J15; footprint (none) -> AES_Library:AES-TermBlock-2POS-5mm-Horz
- J4: renamed from J9; footprint (none) -> AES_Library:AES-CUI_PJ-037B
- J6: renamed from J?; footprint (none) -> AES_Library:PinHeader_2x02_AB-AES; Function CTC Trig SEL -> CTC TRIG; OPT-A (none) -> BCLK; OPT-B (none) -> BCLK/2
- J8: renamed from J?; footprint (none) -> Connector_IDC:IDC-Header_2x20_P2.54mm_Vertical; Function BUS CABLE -> BUS CABLE A; PartOpt1 (none) -> 2x40 Pin HDR
- J9: renamed from J?; footprint (none) -> Connector_IDC:IDC-Header_2x20_P2.54mm_Vertical; Function BUS CABLE -> BUS CABLE B; PartOpt1 (none) -> 2x40 Pin HDR
- M2: renamed from M?; footprint (none) -> AES_Library:OLED-Disp-Socket-P2-8BitPI-AES; PartOpt1 (none) -> 22 SIP Socket; Type1 (none) -> ERMC240128-2 OLED
- R10: renamed from R17; footprint (none) -> Resistor_SMD:R_0805_2012Metric_Pad1.20x1.40mm_HandSolder
- R11: renamed from R19; footprint (none) -> Resistor_SMD:R_0805_2012Metric_Pad1.20x1.40mm_HandSolder
- R12: renamed from R20; footprint (none) -> Resistor_SMD:R_0805_2012Metric_Pad1.20x1.40mm_HandSolder
- R13: renamed from R21; footprint (none) -> Resistor_SMD:R_0805_2012Metric_Pad1.20x1.40mm_HandSolder
- R15: renamed from R13; footprint (none) -> Resistor_SMD:R_0805_2012Metric_Pad1.20x1.40mm_HandSolder
- R16: footprint (none) -> Resistor_SMD:R_0805_2012Metric_Pad1.20x1.40mm_HandSolder
- R17: renamed from R18; footprint (none) -> Resistor_SMD:R_0805_2012Metric_Pad1.20x1.40mm_HandSolder
- R18: renamed from R22; footprint (none) -> Resistor_SMD:R_0805_2012Metric_Pad1.20x1.40mm_HandSolder
- R20: renamed from R?; footprint (none) -> Resistor_SMD:R_0805_2012Metric_Pad1.20x1.40mm_HandSolder
- R6: renamed from R33; footprint (none) -> Resistor_SMD:R_0805_2012Metric_Pad1.20x1.40mm_HandSolder
- R7: renamed from R12; footprint (none) -> Resistor_SMD:R_0805_2012Metric_Pad1.20x1.40mm_HandSolder
- R8: renamed from R14; footprint (none) -> Resistor_SMD:R_0805_2012Metric_Pad1.20x1.40mm_HandSolder
- R9: renamed from R15; footprint (none) -> Resistor_SMD:R_0805_2012Metric_Pad1.20x1.40mm_HandSolder
- RV1: renamed from RV?; footprint (none) -> AES_Library:Pot-Molence-Amazon-PCB-AES
- U31: renamed from U?; value 3.6864MHz OSC -> 3.6864MHz
- U32: renamed from U?; value 74AHC74 -> 74AHCT74DR; footprint (none) -> Package_SO:SOIC-14_3.9x8.7mm_P1.27mm
- U33: renamed from U?6; footprint (none) -> Package_DIP:DIP-28_W15.24mm_LongPads
- U35: renamed from U?7; footprint (none) -> Package_DIP:DIP-40_W15.24mm_Socket_LongPads
- gave numbers to parts that had none: 1
Connections:
- net BA0 is gone; now on net ZA0: U33.18 (CS0), U35.33 (C/~{D})
- net BDRST- is gone; now on net BRDRST-: M1.1 (RESET-), U33.17 (~{RESET}), U35.21 (~{RESET})
- net +3.3V: now also Mod1.22 (3.3V), SD1.4 (VDD), U36.23 (V_{CCB}), U36.24 (V_{CCB}), U?.14 (VCC)
- net +5V: now also J12.18 (5V), J12.58 (5V), J8.18 (Pin_18), J8.38 (Pin_38), M2.20 (BLA/BLK), C4.1, D6.2 (A), J17.19 (Pin_19), J17.2 (Pin_2), SW2.3 (C), U36.1 (V_{CCA}), U37.5 (VCC); no longer J4.1
- net B0IEO: now also J7.2 (Pin_2), U4.12
- net B1IEI: now also J11.1 (Pin_1), U4.11
- net B1IEO: now also J11.2 (Pin_2)
- net BD0: now also J12.27 (D0), J9.7 (Pin_7); no longer U33.25 (D0), U35.40 (D0)
- net BD1: now also J12.28 (D1), J9.8 (Pin_8); no longer U33.26 (D1), U35.1 (D1)
- net BD2: now also J12.29 (D2), J9.9 (Pin_9); no longer U33.27 (D2), U35.39 (D2)
- net BD3: now also J12.30 (D3), J9.10 (Pin_10); no longer U33.28 (D3), U35.2 (D3)
- net BD4: now also J12.31 (D4), J9.11 (Pin_11); no longer U33.1 (D4), U35.38 (D4)
- net BD5: now also J12.32 (D5), J9.12 (Pin_12); no longer U33.2 (D5), U35.3 (D5)
- net BD6: now also J12.33 (D6), J9.13 (Pin_13); no longer U33.3 (D6), U35.37 (D6)
- net BD7: now also J12.34 (D7), J9.14 (Pin_14); no longer U33.4 (D7), U35.4 (D7)
- net BIORQ-: now also J12.26 (~{IORQ}), J9.6 (Pin_6); no longer U33.10 (~{IORQ}), U35.36 (~{IORQ})
- net BRD-: now also J12.25 (~{RD}), J9.5 (Pin_5); no longer U33.6 (~{RD}), U35.32 (~{RD})
- net BWR-: now also J12.24 (~{WR}), J9.4 (Pin_4)
- net CTCIEO: now also U34.2, U5.13
- net EXTIRQ-: now also J13.b1 (Pin_b1), J13.b2 (Pin_b2), J13.b3 (Pin_b3)
- net Earth: now also J20.2 (Pin_2)
- net GND: now also C2.1, J12.17 (GND), J12.57 (GND), J8.17 (Pin_17), J8.37 (Pin_37), M2.21 (BLK/NC), U31.4 (G), U31.7 (G), C4.2, J16.1 (Pin_1), J17.1 (Pin_1), J17.20 (Pin_20), J18.1 (Pin_1), J20.1 (Pin_1), J21.1 (Pin_1), Mod1.24 (GND), Mod1.4 (GND), Mod1.5 (GND), Q1.2 (E), SD1.10 (SHIELD), SD1.6 (VSS), U36.11 (GND), U36.12 (GND), U36.13 (GND), U37.3 (GND), U?.1, U?.10, U?.13, U?.4, U?.7 (GND)
- net MHZ3_7: now also J6.a1 (Pin_a1); no longer J6.a2 (Pin_a2)
- net RXD_A: now also J12.36 (RX), J9.16 (Pin_16)
- net SIOIEO: now also U34.1, U5.12
- net TXD_A: now also J12.35 (TX), J9.15 (Pin_15)
- net ZCLK: now also J12.21 (CLK), J9.1 (Pin_1), J5.a1 (Pin_a1), U11.11 (C); no longer U33.15 (CLK), U35.20 (CLK)
- net ZD0: now also U33.25 (D0), U35.40 (D0), J17.9 (Pin_9), U36.3 (A1)
- net ZD1: now also U33.26 (D1), U35.1 (D1), J17.10 (Pin_10), U36.4 (A2)
- net ZD2: now also U33.27 (D2), U35.39 (D2), J17.11 (Pin_11), U36.5 (A3)
- net ZD3: now also U33.28 (D3), U35.2 (D3), J17.12 (Pin_12), U36.6 (A4)
- net ZD4: now also U33.1 (D4), U35.38 (D4), J17.13 (Pin_13), U36.7 (A5)
- net ZD5: now also U33.2 (D5), U35.3 (D5), J17.14 (Pin_14), U36.8 (A6)
- net ZD6: now also U33.3 (D6), U35.37 (D6), J17.15 (Pin_15), U36.9 (A7)
- net ZD7: now also U33.4 (D7), U35.4 (D7), J17.16 (Pin_16), U36.10 (A8)
- net ZINT-: now also J12.22 (~{INT}), J9.2 (Pin_2)
- net ZM1-: now also J12.19 (~{M1}), J8.19 (Pin_19)
- net at U32.5 (Q): now also J6.a2 (Pin_a2); no longer J6.a1 (Pin_a1)
- net RXD_B: now reaches R11.2
- net RXD_B: now also J12.76 (RX2), J9.36 (Pin_36), J16.2 (Pin_2), Mod1.2 (GPIO0_UTX0)
- net TXD_B: now reaches R12.2
- net TXD_B: now also J12.75 (TX2), J9.35 (Pin_35), J16.3 (Pin_3), Mod1.3 (GPIO1_URX0)
- net BA15: now reaches J8.1 (Pin_1)
- net BA15: now also J12.1 (A15)
- net BA06: now reaches J8.10 (Pin_10)
- net BA06: now also J12.10 (A6)
- net BA05: now reaches J8.11 (Pin_11)
- net BA05: now also J12.11 (A5)
- net BA04: now reaches J8.12 (Pin_12)
- net BA04: now also J12.12 (A4)
- net BA03: now reaches J8.13 (Pin_13)
- net BA03: now also J12.13 (A3)
- net BA02: now reaches J8.14 (Pin_14)
- net BA02: now also J12.14 (A2)
- net BA01: now reaches J8.15 (Pin_15)
- net BA01: now also J12.15 (A1)
- net BA00: now reaches J8.16 (Pin_16)
- net BA00: now also J12.16 (A0)
- net BA14: now reaches J8.2 (Pin_2)
- net BA14: now also J12.2 (A14)
- net BRDRST-: now reaches J8.20 (Pin_20)
- net BRDRST-: now also J12.20 (~{RESET}), M2.9 (~{RST}), J17.8 (Pin_8), U11.13 (~{R}), U?.12
- net CSTM41: now reaches J8.21 (Pin_21)
- net CSTM41: now also J12.41 (CSTM41)
- net CSTM42: now reaches J8.22 (Pin_22)
- net CSTM42: now also J12.42 (CSTM42)
- net CSTM43: now reaches J8.23 (Pin_23)
- net CSTM43: now also J12.43 (CSTM43)
- net CSTM44: now reaches J8.24 (Pin_24)
- net CSTM44: now also J12.44 (CSTM44)
- net CSTM45: now reaches J8.25 (Pin_25)
- net CSTM45: now also J12.45 (CSTM45)
- net CSTM46: now reaches J8.26 (Pin_26)
- net CSTM46: now also J12.46 (CSTM46)
- net CSTM47: now reaches J8.27 (Pin_27)
- net CSTM47: now also J12.47 (CSTM47)
- net CSTM48: now reaches J8.28 (Pin_28)
- net CSTM48: now also J12.48 (CSTM48)
- net BA23: now reaches J8.29 (Pin_29)
- net BA23: now also J12.49 (A23)
- net BA13: now reaches J8.3 (Pin_3)
- net BA13: now also J12.3 (A13)
- net BA22: now reaches J8.30 (Pin_30)
- net BA22: now also J12.50 (A22)
- net BA21: now reaches J8.31 (Pin_31)
- net BA21: now also J12.51 (A21)
- net BA20: now reaches J8.32 (Pin_32)
- net BA20: now also J12.52 (A20)
- net BA19: now reaches J8.33 (Pin_33)
- net BA19: now also J12.53 (A19)
- net BA18: now reaches J8.34 (Pin_34)
- net BA18: now also J12.54 (A18)
- net BA17: now reaches J8.35 (Pin_35)
- net BA17: now also J12.55 (A17)
- net BA16: now reaches J8.36 (Pin_36)
- net BA16: now also J12.56 (A16)
- net ZRFSH-: now reaches J8.39 (Pin_39)
- net ZRFSH-: now also J12.59 (~{RFSH})
- net BA12: now reaches J8.4 (Pin_4)
- net BA12: now also J12.4 (A12)
- net CPURST-: now reaches J8.40 (Pin_40)
- net CPURST-: now also J12.60 (~{CPURST})
- net BA11: now reaches J8.5 (Pin_5)
- net BA11: now also J12.5 (A11)
- net BA10: now reaches J8.6 (Pin_6)
- net BA10: now also J12.6 (A10)
- net BA09: now reaches J8.7 (Pin_7)
- net BA09: now also J12.7 (A9)
- net BA08: now reaches J8.8 (Pin_8)
- net BA08: now also J12.8 (A8)
- net BA07: now reaches J8.9 (Pin_9)
- net BA07: now also J12.9 (A7)
- net BD_OPT1-: now reaches U35.23 (~{CTSB})
- net BD_OPT1-: now also J18.2 (Pin_2), J19.b3 (Pin_b3)
- net CONPWR: now reaches R20.1
- net CONPWR: now also M2.19 (VEE/BLA), J17.18 (Pin_18); no longer M2.20 (BLA/BLK)
- net DISP_BL-: now reaches R18.2
- net CONV0: now reaches M2.4 (V0), RV1.2
- net CONV0: now also J17.3 (Pin_3)
- net ZWR-: now reaches M2.5 (~{WR})
- net ZWR-: now also J17.4 (Pin_4), U?.9
- net ZRD-: now reaches M2.6 (~{RD})
- net ZRD-: now also U33.6 (~{RD}), U35.32 (~{RD}), J17.5 (Pin_5), U36.2 (A>B)
- net DISPSEL-: now reaches M2.7 (~{CE})
- net DISPSEL-: now also J17.6 (Pin_6)
- net ZA0: now reaches M2.8 (C/~{D})
- net ZA0: now also J17.7 (Pin_7), U?.5
- net BMREQ-: now reaches J12.23 (~{MREQ})
- net BMREQ-: now also J9.3 (Pin_3)
- net USR1: now reaches J12.37 (User1)
- net USR1: now also J9.17 (Pin_17), J13.a1 (Pin_a1)
- net USR2: now reaches J12.38 (User2)
- net USR2: now also J9.18 (Pin_18), J13.a2 (Pin_a2)
- net USR3: now reaches J12.39 (User3)
- net USR3: now also J9.19 (Pin_19), J13.a3 (Pin_a3)
- net IOCLK: now reaches J12.61 (CLK2)
- net IOCLK: now also J9.21 (Pin_21), U33.15 (CLK), U35.20 (CLK), J5.b1 (Pin_b1), J5.b2 (Pin_b2)
- net ZBSAK-: now reaches J12.62 (~{BSACK})
- net ZBSAK-: now also J9.22 (Pin_22)
- net ZHALT-: now reaches J12.63 (~{HALT})
- net ZHALT-: now also J9.23 (Pin_23)
- net ZBREQ-: now reaches J12.64 (~{BSREQ})
- net ZBREQ-: now also J9.24 (Pin_24)
- net ZWAIT-: now reaches J12.65 (~{WAIT})
- net ZWAIT-: now also J9.25 (Pin_25), Q1.3 (C)
- net ZNMI-: now reaches J12.66 (~{NMI})
- net ZNMI-: now also J9.26 (Pin_26)
- net NC_D08: now reaches J12.67 (D8)
- net NC_D08: now also J9.27 (Pin_27)
- net NC_D09: now reaches J12.68 (D9)
- net NC_D09: now also J9.28 (Pin_28)
- net NC_D10: now reaches J12.69 (D10)
- net NC_D10: now also J9.29 (Pin_29)
- net NC_D11: now reaches J12.70 (D11)
- net NC_D11: now also J9.30 (Pin_30)
- net NC_D12: now reaches J12.71 (D12)
- net NC_D12: now also J9.31 (Pin_31)
- net NC_D13: now reaches J12.72 (D13)
- net NC_D13: now also J9.32 (Pin_32)
- net NC_D14: now reaches J12.73 (D14)
- net NC_D14: now also J9.33 (Pin_33)
- net NC_D15: now reaches J12.74 (D15)
- net NC_D15: now also J9.34 (Pin_34)
- net USR5: now reaches J12.77 (User5)
- net USR5: now also J9.37 (Pin_37), J19.a1 (Pin_a1)
- net USR6: now reaches J12.78 (User6)
- net USR6: now also J9.38 (Pin_38), J19.a2 (Pin_a2)
- net USR7: now reaches J12.79 (User7)
- net USR7: now also J9.39 (Pin_39), J19.a3 (Pin_a3)
- net BA1 renamed ZA1
- net FONT_BL renamed FONT1
- net FONT1: now also J17.17 (Pin_17)
- net LCLIEO renamed LCLIA-
- net LCLIA-: now also J7.1 (Pin_1), U4.13, U5.11
- net VPU? renamed VPU1
- net VPU1: now also U11.10 (~{S})
- net VPU?0 renamed VPU2
- new net: J4.1, SW2.2 (B)
- new net: J5.a2 (Pin_a2), U11.9 (Q)
- new net: U11.12 (D), U11.8 (~{Q})
- new net: Q1.1 (B), R19.2
- new net BUSIA-: U34.12
- new net INTACK: U34.13
- new net MA0: Mod1.21 (GPIO29_A3), U?.6
- new net MRST-: Mod1.23 (RESET), U?.11
- new net MWR-: Mod1.20 (GPIO28_A2), U?.8
- new net SDCS-: Mod1.14 (GPIO10_PWM5A), SD1.2 (DAT3/CD)
- new net SPICK: Mod1.17 (GPIO18_SCK0), SD1.5 (CLK)
- new net SPIMI: Mod1.16 (GPIO20_MISO0), SD1.7 (DAT0)
- new net SPIMO: Mod1.15 (GPIO19_MOSI0), SD1.3 (CMD)
- new net UHPWR5: D6.1 (K), Mod1.25 (5V_RAW)
- new net USBD+: J21.2 (Pin_2), Mod1.1 (D+)
- new net USBD-: J21.3 (Pin_3), Mod1.26 (D-)
- new net USBSDSEL-: Mod1.19 (GPIO27_A1), U36.22 (~{OE}), U37.2, U?.2, U?.3
- new net V3D0: Mod1.6 (GPIO2_SDA1), U36.21 (B1)
- new net V3D1: Mod1.7 (GPIO3_SCL1), U36.20 (B2)
- new net V3D2: Mod1.8 (GPIO4_UTX1), U36.19 (B3)
- new net V3D3: Mod1.9 (GPIO5_URX1), U36.18 (B4)
- new net V3D4: Mod1.10 (GPIO6_PWM3A), U36.17 (B5)
- new net V3D5: Mod1.11 (GPIO7_PWM3B), U36.16 (B6)
- new net V3D6: Mod1.12 (GPIO8_PWM4A), U36.15 (B7)
- new net V3D7: Mod1.13 (GPIO9_PWM4B), U36.14 (B8)
- new net WAIT: R19.1, U37.4
- new net WAITRQ-: Mod1.18 (GPIO26_A0), U37.1
- new net ZIORQ-: U33.10 (~{IORQ}), U35.36 (~{IORQ})
- no-connect marks 4 -> 12
Other:
- note added: "1x22 Socket for Display Module or 2x10 Pin Header (for Ribbon Cable, w/Module pins 1&22 NC)"
- note added: "KBD"
- note added: "Module provides 3.3V"
- moved on the sheet: C2, C3, C5, C6, J10, J12, J14, J15, J3, J4, J6, J8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

Commit message: ZMB: v1.0 Board RFP
Parts:
- removed J10, J19: Conn_02x03, AES_Library:PinHeader_2x03_AB-AES, symbol Connector_Generic:Conn_02x03_Row_Letter_First
- removed J11, J18, J20, J7: HDR 1x02 Pin, Connector_PinHeader_2.54mm:PinHeader_1x02_P2.54mm_Vertical, symbol Connector_Generic:Conn_01x02
- removed J13: HDR 02x03 PIN, AES_Library:PinHeader_2x03_AB-AES, symbol Connector_Generic:Conn_02x03_Row_Letter_First
- removed J14: CONN 02x05 - DTE_HDR-AES, AES_Library:AES-PinHeader_2x05_DB9-Order, symbol AES_Library:DTE_HDR-AES
- removed J15: Conn_02x05 HDR, AES_Library:PinHeader_2x05_AB-AES, symbol Connector_Generic:Conn_02x05_Row_Letter_First
- removed J21: HDR 1x3 Pin, Connector_PinHeader_2.54mm:PinHeader_1x03_P2.54mm_Vertical, symbol Connector_Generic:Conn_01x03
- removed J3: Screw_Terminal_01x02, AES_Library:AES-TermBlock-2POS-5mm-Horz, symbol Connector:Screw_Terminal_01x02
- removed J5, J6: HDR 02x02, AES_Library:PinHeader_2x02_AB-AES, symbol Connector_Generic:Conn_02x02_Row_Letter_First
- removed Mod1: Adafruit KB2040 Module, AES_Library:Adafruit-KB2040-AES, symbol AES_Library:Adafruit-KB2040-AES
- removed Q1: MMBT3904, Package_TO_SOT_SMD:SOT-23, symbol Transistor_BJT:MMBT3904
- removed R19: 100, Resistor_SMD:R_0805_2012Metric_Pad1.20x1.40mm_HandSolder, symbol Device:R_Small_US
- removed U11, U32: 74AHCT74DR, Package_SO:SOIC-14_3.9x8.7mm_P1.27mm, symbol 74xx:74HC74
- removed U?: 74LVC125, symbol 74xx:74LVC125
- added C38, C39, C41, C42, C43: 1.0uF, Capacitor_SMD:C_0603_1608Metric, symbol Device:C_Small
- added C4: 220uF, Capacitor_THT:CP_Radial_D6.3mm_P2.50mm, symbol Device:C_Polarized_Small_US
- added J10, J14: HDR 1x04 Socket, Connector_PinSocket_2.54mm:PinSocket_1x04_P2.54mm_Vertical, symbol Connector_Generic:Conn_01x04
- added J18: DE9 Male (PINS), AES_Library:DSUB9-Pins-AdamTech_DE09-PL-25-AES, symbol Connector:DE9_Pins
- added J3: HDR 1x02 Pin, Connector_PinHeader_2.54mm:PinHeader_1x02_P2.54mm_Vertical, symbol Connector_Generic:Conn_01x02
- added JP1, JP2, JP3, JP4: CONN 1x02 HDR Pins 2mm, Connector_PinHeader_2.00mm:PinHeader_1x02_P2.00mm_Vertical, symbol Jumper:Jumper_2_Open
- added JP5, JP6, OP8: HDR 1x02 Pin, Connector_PinHeader_2.00mm:PinHeader_1x02_P2.00mm_Vertical, symbol Connector_Generic:Conn_01x02
- added OP2, OP3: AES-Option_A-B, Connector_PinHeader_2.00mm:PinHeader_1x03_P2.00mm_Vertical, symbol AES_Library:AES-Option_A-B
- added OP6: CONN 2x3 HDR, AES_Library:PinHeader_2x03_AB_2mm-AES, symbol Connector_Generic:Conn_02x03_Row_Letter_First
- added OP7: HDR 2x02 2mm, AES_Library:PinHeader_2x02_AB_2mm-AES, symbol Connector_Generic:Conn_02x02_Row_Letter_First
- added Q1: DMG2305UX, AES_Library:DMG2305-SOT-23-3-AES, symbol AES_Library:DMG2305UX-AES
- added R22, R28, R30, R31, R32, R33: 10k, Resistor_SMD:R_0805_2012Metric, symbol Device:R_Small_US
- added R23, R24, R25: 20k, Resistor_SMD:R_0805_2012Metric, symbol Device:R_Small_US
- added R27: 0, Resistor_SMD:R_0805_2012Metric, symbol Device:R_Small_US
- added R29: 33.2k, Resistor_SMD:R_0805_2012Metric, symbol Device:R_Small_US
- added U39: 74AHCT04, Package_SO:SOIC-14_3.9x8.7mm_P1.27mm, symbol AES_Library:7404-AES
- added unit 1 of U43
- added U45: WS-RP2040-Zero, AES_Library:RP2040_WS-ZERO-AES, symbol AES_Library:RP2040_WS-AES
- added U46: MAX232/ST232, Package_SO:SOIC-16_3.9x9.9mm_P1.27mm, symbol AES_Library:MAX232-ST232-AES
- added U47: 74LVC1G06W, Package_TO_SOT_SMD:SOT-23-5, symbol AES_Library:74LVC1G06-AES
- C2, C5: footprint Capacitor_SMD:C_0603_1608Metric_Pad1.08x0.95mm_HandSolder -> Capacitor_SMD:C_0603_1608Metric
- D6: value CDBF0130R -> PMEG2010AEB; footprint Diode_SMD:D_SOD-323F -> Diode_SMD:D_SOD-323_HandSoldering; Spec 30V 100MA SCHTK -> SCHOTTKY 40V
- J12: Function BP80 BUS (1) -> RCBus-Z80 (0)
- J8: Function BUS CABLE A -> Backplane CBL A
- J9: Function BUS CABLE B -> Backplane CBL B
- M1: Function (none) -> COM2
- R10, R11, R12, R13, R15, R16, R18, R6, R7, R9: footprint Resistor_SMD:R_0805_2012Metric_Pad1.20x1.40mm_HandSolder -> Resistor_SMD:R_0805_2012Metric
- R17, R8: value 22 -> 10k; footprint Resistor_SMD:R_0805_2012Metric_Pad1.20x1.40mm_HandSolder -> Resistor_SMD:R_0805_2012Metric
- R20: value 180 -> 7.5k; footprint Resistor_SMD:R_0805_2012Metric_Pad1.20x1.40mm_HandSolder -> Resistor_SMD:R_0805_2012Metric
- RV1: Function (none) -> CONTRAST
- SW2: symbol Switch:SW_SPDT -> AES_Library:SW_SPDT-TGL-PCMount-AES
- U31: value 3.6864MHz -> 3.6864MHz Can Osc; footprint Package_DIP:DIP-14_W7.62mm_LongPads -> AES_Library:OSC-8_14-AES; Freq 12MHz -> 3.6864MHz
- U34: value 74AHCT10 -> 74ACT10
- U43: renamed from U?; value 74LVC125 -> 74LVC125AS; footprint (none) -> Package_SO:SOIC-14_3.9x8.7mm_P1.27mm
- renumbered C4 to C44
Connections:
- net DCD_A is gone; now on net +5V: R17.2
- net DISP_BL- is gone; now on net FONT1: R18.2
- net MHZ3_7 is gone; now on net CTC_CLK: U31.11 (O), U31.8 (O), U33.22 (CLK/TRG1), U33.23 (CLK/TRG0)
- net MRST- is gone; now on net MWR-: U43.11
- net RI_A is gone; now on net CNSLSELB-: R8.2
- net USR1 is gone; now on net ExIRQ1-: J12.37 (~{zIRQ1}), J9.17 (Pin_17)
- net USR5 is gone; now on net ExIRQ2-: J12.77 (~{zINT2}), J9.37 (Pin_37)
- net ZNMI- is gone; now on net NMIREQ-: J12.66 (~{NMI}), J9.26 (Pin_26)
- net +3.3V: now also J10.1 (Pin_1), R23.1, R30.2, R31.2, R32.2, R33.2, U45.21 (3V3)
- net +5V: now also R8.1, C39.1, C4.1, C41.2, JP5.2 (Pin_2), Q1.2 (S), R22.1, R25.1, R27.1, R28.2, U46.16 (VCC), U47.5 (VCC); no longer D6.2 (A), J17.19 (Pin_19), M2.20 (BLA/BLK)
- net B0IEO: now also J12.39 (IEO), JP4.2 (B); no longer J9.20 (Pin_20)
- net BRDRST-: no longer U43.12
- net CTC2_OUT: now also OP7.a1 (Pin_a1)
- net CTC3_CLK: now also OP7.b1 (Pin_b1), OP7.b2 (Pin_b2)
- net FONT1: no longer R13.2
- net GND: now also C39.2, C4.2, C43.1, J10.2 (Pin_2), J18.5, J3.1 (Pin_1), OP8.1 (Pin_1), R24.2, R29.2, U43.1, U45.22 (GND), U46.15 (GND), U47.3 (GND); no longer RV1.1
- net IOCLK: now also OP6.b1 (Pin_b1), OP6.b2 (Pin_b2), OP6.b3 (Pin_b3)
- net LCLIA-: now also J12.38 (IEI), JP4.1 (A); no longer J9.40 (Pin_40)
- net MA0: now also U45.11 (GP10)
- net MWR-: now also U45.13 (GP12); no longer U43.8
- net RXD_A: no longer R7.2
- net RXD_B: no longer J16.2 (Pin_2), R11.2
- net SDCS-: now also R30.1, U45.20 (GP29)
- net SPICK: now also R33.1, U45.17 (GP26)
- net SPIMI: now also R32.1, U45.19 (GP28)
- net SPIMO: now also R31.1, U45.18 (GP27)
- net TXD_A: no longer R15.2
- net TXD_B: no longer J16.3 (Pin_3), R12.2
- net UHPWR5: now also U45.23 (VBUS)
- net USBSDSEL-: now also U43.2
- net V3D0: now also U45.3 (GP2)
- net V3D1: now also U45.4 (GP3)
- net V3D2: now also U45.5 (GP4)
- net V3D3: now also U45.6 (GP5)
- net V3D4: now also U45.7 (GP6)
- net V3D5: now also U45.8 (GP7)
- net V3D6: now also U45.9 (GP8)
- net V3D7: now also U45.10 (GP9)
- net WAIT: now also U47.2
- net WAITRQ-: now also R23.2, U45.15 (GP14)
- net ZCLK: now also OP6.a1 (Pin_a1)
- net ZRD-: now also U43.9
- net ZWAIT-: now also U47.4
- net ZWR-: now also U43.12; no longer U43.9
- net +5IN: now reaches J4.1, SW2.2 (B)
- net CNSLSELB-: now reaches U35.11 (~{SYNCA})
- net CNSLSELB-: now also OP8.2 (Pin_2); no longer R8.1
- net at R7.1: now also U46.14 (T1OUT); no longer U35.12 (RxDA)
- net at R15.1: now also U46.7 (T2OUT); no longer U35.15 (TxDA)
- net at R9.1: now also U46.13 (R1IN); no longer U35.17 (~{RTSA})
- net at R16.1: now also U46.8 (R2IN); no longer U35.18 (~{CTSA})
- net ExIRQ1-: now reaches U35.19 (~{DCDA})
- net ExIRQ1-: now also R6.1; no longer R17.1
- net at M1.7 (TXD(O)): now also JP6.2 (Pin_2)
- net CHB_TXD: now reaches M1.9 (RXD(I))
- net CHB_TXD: now also J16.3 (Pin_3), R12.2
- net B1IEI renamed USR8
- net USR8: now also J9.40 (Pin_40), JP1.2 (B); no longer U4.11
- net B1IEO renamed CRSTRQ-
- net CRSTRQ-: now also J9.20 (Pin_20)
- net BD_OPT1- renamed MODIRQ-
- net MODIRQ-: now also U39.12
- net CPURST- renamed RCBPAGE
- net CSTM42 renamed BAI0
- net BAI0: now also JP3.1 (A), R28.1; no longer J8.22 (Pin_22)
- net CSTM43 renamed BAO0
- net BAO0: now also J8.22 (Pin_22), JP3.2 (B); no longer J8.23 (Pin_23)
- net CTC_CLK2 renamed CTC_CLK
- net CTC_CLK: now also OP7.a2 (Pin_a2)
- net CTS_A renamed HSIN
- net HSIN: now also OP3.2 (C)
- net DTR_A renamed CHA_DTR-
- net CHA_DTR-: now also J3.2 (Pin_2)
- net EXTIRQ- renamed ExIRQ2-
- net ExIRQ2-: now also R17.1; no longer R6.1
- net RTS_A renamed C1_RXD
- net C1_RXD: now also J18.2
- net USR2 renamed bpIEI
- net bpIEI: now also U4.11, JP2.1 (A); no longer J12.38 (User2)
- net USR3 renamed bpIEO
- net bpIEO: now also JP2.2 (B); no longer J12.39 (User3)
- net VPU2: no longer names the net of U35.6 (IEI)
- net VPU2: now also R22.2
- new net: C38.1, U46.1 (C1+)
- new net: C41.1, U46.2 (VS+)
- new net: C38.2, U46.3 (C1-)
- new net: C42.2, U46.4 (C2+)
- new net: C42.1, U46.5 (C2-)
- new net: C43.2, U46.6 (VS-)
- new net: D6.2 (A), JP5.1 (Pin_1), R27.2
- new net: R29.1, RV1.1
- new net BAObp: J8.23 (Pin_23)
- new net BLPWR: J17.19 (Pin_19), M2.20 (BLA/BLK), Q1.3 (D)
- new net C1_CTS: J18.8, OP3.1 (A)
- new net C1_DSR: J18.6, OP3.3 (B)
- new net C1_DTR: J18.4, OP2.3 (B)
- new net C1_RTR: J18.7, OP2.1 (A)
- new net C1_TXD: J18.3, R7.2
- new net CHA_CTS-: U35.18 (~{CTSA}), U46.9 (R2OUT)
- new net CHA_RTR-: U35.17 (~{RTSA}), U46.10 (T2IN)
- new net CHA_RXD: U35.12 (RxDA), U46.12 (R1OUT)
- new net CHA_TXD: U35.15 (TxDA), U46.11 (T1IN)
- new net CHB_RXD: J16.2 (Pin_2), JP6.1 (Pin_1), R11.2
- new net CLKf: OP6.a2 (Pin_a2)
- new net CLKh: OP6.a3 (Pin_a3)
- new net DSPBLON-: Q1.1 (G), R25.2
- new net HSOUT: OP2.2 (C), R15.2
- new net INTRQ: R24.1, U39.13, U45.16 (GP15)
- new net MRD-: U43.8, U45.12 (GP11)
- new net MSEL-: U43.3, U45.14 (GP13)
- new net SCL0_RX: J10.3 (Pin_3), U45.2 (GP1)
- new net SDA_TX: J10.4 (Pin_4), U45.1 (GP0)
- new net USR8J: JP1.1 (A), R13.2
- no-connect marks 12 -> 18
Other:
- note added: "3.3V Logic Section"
- note added: "NOTE: Configure module for 5V operation"
- note added: "NOTE: DCE (USB) to DTE (ZMB)"
- note removed: "NOTE: DCE (USB) to DTE (Board)"
- moved on the sheet: C44, C5, C6, D6, J16, J17, M1, M2, R10, R11, R12, R13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
