File: hw/SD-ZMB/logic_pwr_spr.kicad_sch (KiCad schematic)
At the start: 50 parts

Commit message: PR7.4: checkpoint only
Parts:
- added U? (x2): 74HC04, symbol AES_Library:7404-AES
- added U? (x3): 74HC02, symbol 74xx:74HC02
