File: hw/SD-ZMB/mainboard.kicad_sch (KiCad schematic)
At the start: 60 parts

Commit message: PR7: Review
Parts:
- removed RN? (x5): 10k, Resistor_THT:R_Array_SIP9, symbol Device:R_Network08_US
- removed U? (x7): 74AHC08, symbol 74xx:74LS08
- removed U? (x2): 74HCT08, symbol 74xx:74LS08
- removed U?: 74HC245-AES, symbol AES_Library:74HC245-AES
- removed U? (x5): 74HCT14, symbol AES_Library:74HC14-AES
- removed U? (x2): 74HCT00, symbol 74xx:74HC00
- removed U?: 74AHC14, symbol AES_Library:74HC14-AES
- removed U?: AS6C4008, Package_DIP:DIP-32_W15.24mm, symbol Memory_RAM:AS6C4008-55PCN
- removed U? (x2): 74AHC138, symbol 74xx:74HC138
- removed U?: 74HCT32, symbol 74xx:74LS32
- removed U?: 74AHC245, symbol AES_Library:74HC245_BA-AES
- removed U?: SST39SF040, symbol AES_Library:Flash-SST39SF0n0-AES
- removed U? (x2): 74HCT86, symbol 74xx:74LS86
- removed U? (x2): 74AHC245, symbol AES_Library:74HC245-AES
- removed U?: 8K/32K SRAM, Package_DIP:DIP-28_W7.62mm, symbol AES_Library:SRAM-Cache-8K32K-A-EAS
- added RN? (x3): 20k, Resistor_THT:R_Array_SIP9, symbol Device:R_Network08_US
- added RN? (x2): 10k, Resistor_THT:R_Array_SIP9, symbol Device:R_Network08_US
- added U? (x7): 74AHC08, symbol 74xx:74LS08
- added U?: 74HCT08, symbol 74xx:74LS08
- added U?: SST39SF040, symbol AES_Library:Flash-SST39SF0n0-AES
- added U?: 74AHC245, symbol AES_Library:74HC245_BA-AES
- added U? (x3): 74HCT00, symbol 74xx:74HC00
- added U? (x5): 74HCT14, symbol AES_Library:74HC14-AES
- added U? (x2): 74HCT86, symbol 74xx:74LS86
- added U? (x4): 74AHC245, symbol AES_Library:74HC245-AES
- added U? (x2): 74AHC138, symbol 74xx:74HC138
- added U?: 74HCT32, symbol 74xx:74LS32
- added U?: 74AHC14, symbol AES_Library:74HC14-AES
- added U?: 74AHC541-AES, symbol AES_Library:74AHC541-AES
- added U?: AS6C4008, Package_DIP:DIP-32_W15.24mm, symbol Memory_RAM:AS6C4008-55PCN
- added U?: 8K/32K SRAM, Package_DIP:DIP-28_W7.62mm, symbol AES_Library:SRAM-Cache-8K32K-A-EAS
Connections:
- net +5V: now also RN?.1 (common), RN?.1 (common), U?.16 (VCC), U?.16 (VCC), U?.20 (VCC), U?.20 (VCC), U?.20 (VCC), U?.20 (VCC), U?.20 (VCC), U?.20 (VCC), U?.28 (V_{CC}), U?.32 (VCC), U?.32 (VCC)
- net BDRST-: now also U?.1
- net CPURST-: now also U?.2
- net GND: now also RN?.1 (common), RN?.1 (common), RN?.1 (common), U?.1 (A14/NC), U?.10 (GND), U?.10 (GND), U?.10 (GND), U?.10 (GND), U?.10 (GND), U?.10 (GND), U?.14 (GND), U?.16 (GND), U?.16 (VSS), U?.19 (~{OE}), U?.19 (~{OE}), U?.19 (~{OE}), U?.2 (A_{12}), U?.20 (~{CE_{1}}), U?.21 (A_{10}), U?.23 (A_{11}), U?.24 (A_{9}), U?.25 (A_{8}), U?.3 (A_{7}), U?.4 (A_{6}), U?.5 (A_{5}), U?.6 (A_{4}), U?.7 (A5), U?.8 (A6), U?.8 (GND), U?.8 (GND), U?.9 (A7)
- net LOCALOP-: now also U?.4
- net MEM_OP-: now also U?.4 (~{E0}), U?.4 (~{E0})
- net NMI-: now also U?.8
- net NMIEN: now also U?.1
- net PDA16: now also U?.5 (A3)
- net PDA17: now also U?.6 (A4)
- net PDA18: now also U?.7 (A5)
- net PDA19: now also U?.8 (A6)
- net PDA20: now also U?.9 (A7)
- net PGINGEN: now also U?.1, U?.13, U?.6 (E2)
- net PGRGRD-: now also U?.5
- net PGRGSEL-: now also U?.1, U?.19 (~{OE})
- net PGRGWR-: now also U?.1 (A>B), U?.27 (~{WE})
- net PRA3: now also U?.3, U?.7 (A_{3})
- net PROE-: now also U?.22 (~{OE}), U?.6
- net RA55RO: now also U?.3 (A2)
- net RAMRD-: now also U?.24 (OE#), U?.6
- net RAMRDP-: now also U?.10 (~{Y5}), U?.5
- net RAMRDZ-: now also U?.10 (~{Y5}), U?.4
- net RAMWR-: now also U?.29 (WE#), U?.6
- net RAMWRP-: now also U?.5, U?.9 (~{Y6})
- net RAMWRZ-: now also U?.4, U?.9 (~{Y6})
- net ROMRD-: now also U?.24 (OE#), U?.6
- net ROMRDP-: now also U?.14 (~{Y1}), U?.5
- net ROMRDZ-: now also U?.14 (~{Y1}), U?.4
- net ROMWR-: now also U?.31 (PGM#), U?.6
- net ROMWRP-: now also U?.13 (~{Y2}), U?.5
- net ROMWRZ-: now also U?.13 (~{Y2}), U?.4
- net VPU?: now also U?.26 (A13/CE_{2})
- net ZA0: now also U?.1, U?.12 (A0), U?.12 (A0), U?.2 (A0)
- net ZA1: now also U?.11 (A1), U?.11 (A1), U?.3 (A1)
- net ZA10: now also U?.23 (A10), U?.23 (A10), U?.4 (A2)
- net ZA11: now also U?.25 (A11), U?.25 (A11), U?.5 (A3)
- net ZA12: now also U?.4 (A12), U?.4 (A12), U?.6 (A4)
- net ZA13: now also U?.10 (A_{0}), U?.2 (A0)
- net ZA14: now also U?.3 (A1), U?.9 (A_{1})
- net ZA15: now also U?.4 (A2), U?.8 (A_{2})
- net ZA2: now also U?.10 (A2), U?.10 (A2), U?.4 (A2)
- net ZA3: now also U?.5 (A3), U?.9 (A3), U?.9 (A3)
- net ZA4: now also U?.6 (A4), U?.8 (A4), U?.8 (A4)
- net ZA5: now also U?.7 (A5), U?.7 (A5), U?.7 (A5)
- net ZA6: now also U?.6 (A6), U?.6 (A6), U?.8 (A6)
- net ZA7: now also U?.5 (A7), U?.5 (A7), U?.9 (A7)
- net ZA8: now also U?.2 (A0), U?.27 (A8), U?.27 (A8)
- net ZA9: now also U?.26 (A9), U?.26 (A9), U?.3 (A1)
- net ZBNIO-: now also U?.3, U?.4
- net ZBSAK-: now also U?.1
- net ZD0: now also RN?.2 (R1), U?.13 (D0), U?.13 (DQ0), U?.18 (B0), U?.2 (A0)
- net ZD1: now also RN?.3 (R2), U?.14 (D1), U?.14 (DQ1), U?.17 (B1), U?.3 (A1)
- net ZD2: now also RN?.4 (R3), U?.15 (D2), U?.15 (DQ2), U?.16 (B2), U?.4 (A2)
- net ZD3: now also RN?.5 (R4), U?.15 (B3), U?.17 (D3), U?.17 (DQ3), U?.5 (A3)
- net ZD4: now also RN?.6 (R5), U?.14 (B4), U?.18 (D4), U?.18 (DQ4), U?.6 (A4)
- net ZD5: now also RN?.7 (R6), U?.13 (B5), U?.19 (D5), U?.19 (DQ5), U?.7 (A5)
- net ZD6: now also RN?.8 (R7), U?.12 (B6), U?.20 (D6), U?.20 (DQ6), U?.8 (A6)
- net ZD7: now also RN?.9 (R8), U?.11 (B7), U?.21 (D7), U?.21 (DQ7), U?.9 (A7)
- net ZDIN-: now also U?.2, U?.2 (A1), U?.2 (A1), U?.3, U?.5
- net ZIORQ: now also U?.12, U?.2, U?.22 (CE#), U?.22 (CE#)
- net ZIORQ-: now also U?.13, U?.2
- net ZM1-: now also U?.2
- net ZMASTER: now also U?.1, U?.1 (A>B), U?.1 (A>B), U?.2
- net ZNMI-: now also U?.9
- net ZRD-: now also U?.1
- net ZRST: now also U?.2
- net ZRST-: now also U?.1, U?.3
- net ZWR-: now also U?.1 (A0), U?.1 (A0)
- new net: U?.1, U?.2 (x2)
- new net: U?.2, U?.3
- new net: U?.10, U?.2
- new net: U?.19 (~{OE}), U?.6
- new net BA00: RN?.2 (R1), U?.18 (B0)
- new net BA01: RN?.3 (R2), U?.17 (B1)
- new net BA02: RN?.4 (R3), U?.16 (B2)
- new net BA03: RN?.5 (R4), U?.15 (B3)
- new net BA04: RN?.6 (R5), U?.14 (B4)
- new net BA05: RN?.7 (R6), U?.13 (B5)
- new net BA06: RN?.8 (R7), U?.12 (B6)
- new net BA07: RN?.9 (R8), U?.11 (B7)
- new net BA08: RN?.2 (R1), U?.18 (B0)
- new net BA09: RN?.3 (R2), U?.17 (B1)
- new net BA10: RN?.4 (R3), U?.16 (B2)
- new net BA11: RN?.5 (R4), U?.15 (B3)
- new net BA12: RN?.6 (R5), U?.14 (B4)
- new net BA13: RN?.7 (R6), U?.13 (B5)
- new net BA14: RN?.8 (R7), U?.12 (B6)
- new net BA15: RN?.9 (R8), U?.11 (B7)
- new net BA16: RN?.2 (R1), U?.18 (B0)
- new net BA17: RN?.3 (R2), U?.17 (B1)
- new net BA18: RN?.4 (R3), U?.16 (B2)
- new net BA19: RN?.5 (R4), U?.15 (B3)
- new net BA20: RN?.6 (R5), U?.14 (B4)
- new net BA21: RN?.7 (R6), U?.13 (B5)
- new net BA22: RN?.8 (R7), U?.12 (B6)
- new net BA23: RN?.9 (R8), U?.11 (B7)
- new net BD0: RN?.2 (R1), U?.18 (B0)
- new net BD1: RN?.3 (R2), U?.17 (B1)
- new net BD2: RN?.4 (R3), U?.16 (B2)
- new net BD3: RN?.5 (R4), U?.15 (B3)
- new net BD4: RN?.6 (R5), U?.14 (B4)
- new net BD5: RN?.7 (R6), U?.13 (B5)
- new net BD6: RN?.8 (R7), U?.12 (B6)
- new net BD7: RN?.9 (R8), U?.11 (B7)
- new net LMA13: U?.11 (I/O_{1}), U?.18 (Y0), U?.2 (A0), U?.28 (A13), U?.28 (A13), U?.7 (A5)
- new net LMA14: U?.12 (I/O_{2}), U?.17 (Y1), U?.29 (A14), U?.3 (A1), U?.3 (A14), U?.8 (A6)
- new net LMA15: U?.13 (I/O_{3}), U?.16 (Y2), U?.3 (A15), U?.31 (A15), U?.4 (A2), U?.9 (A7)
- new net LMA16: U?.15 (I/O_{4}), U?.15 (Y3), U?.2 (A0), U?.2 (A16), U?.2 (A16), U?.5 (A3)
- new net LMA17: U?.14 (Y4), U?.16 (I/O_{5}), U?.3 (A1), U?.30 (A17), U?.30 (A17), U?.6 (A4)
- new net LMA18: U?.1 (A18), U?.1 (A18), U?.13 (Y5), U?.17 (I/O_{6}), U?.4 (A2), U?.7 (A5)
- new net LMA19: U?.12 (Y6), U?.18 (I/O_{7}), U?.3 (A2), U?.5 (A3), U?.8 (A6)
- new net LMA20: U?.11 (Y7), U?.19 (I/O_{8}), U?.5 (~{E1}), U?.5 (~{E1}), U?.6 (A4), U?.9 (A7)
- new net NOPAGE: U?.12, U?.6 (E2)
- new net ZDTOBD: U?.1 (A>B), U?.3
- new net ZPGPRS-: U?.1 (~{G1}), U?.19 (~{G2}), U?.3
Other:
- moved on the sheet: OPT?, RN?, U?, U?A, U?B, U?D

Commit message: PR7.4: checkpoint only
Parts:
- removed C?: 22uf, symbol Device:C
- removed D?: 1N4148, Diode_THT:D_DO-35_SOD27_P7.62mm_Horizontal, symbol Diode:1N4148
- removed J?: Conn_01x02, symbol Connector_Generic:Conn_01x02
- removed SW?: SW_Push, symbol Switch:SW_Push
- removed U? (x6): 74AHC08, symbol 74xx:74LS08
- removed U?: 74HC4002, symbol 4xxx:4002
- removed U? (x5): 74HCT14, symbol AES_Library:74HC14-AES
- removed U? (x2): 74HCT86, symbol 74xx:74LS86
- removed U? (x2): 74AHC138, symbol 74xx:74HC138
- removed U? (x3): 74AHC245, symbol AES_Library:74HC245-AES
- removed U?: 74HCT08, symbol 74xx:74LS08
- removed U? (x2): 74HCT32, symbol 74xx:74LS32
- removed U?: 74AHC14, symbol AES_Library:74HC14-AES
- added SW?: SW Push (4 pin), symbol AES_Library:SW_Push_Tactile_12-34
- added U? (x2): 74HC243, symbol AES_Library:74HC243-AES
- added U? (x6): 74HC04, symbol AES_Library:7404-AES
- added U? (x10): 74AHC08, symbol 74xx:74LS08
- added U? (x9): 74HCT00, symbol 74xx:74HC00
- added U?: 74HCT08, symbol 74xx:74LS08
- added U? (x3): 74AHC245, symbol AES_Library:74245-AES
- added U? (x2): 74HC4002, symbol 4xxx:4002
- added U? (x5): 74HCT32, symbol 74xx:74LS32
- added U?: MIC2775, Package_TO_SOT_SMD:SOT-23-5, symbol AES_Library:MIC2775-AES
- added U? (x2): 74HCT86, symbol 74xx:74LS86
- added U? (x2): 74HC02, symbol 74xx:74HC02
- added U? (x2): 74HCT02, symbol 74xx:74HC02
- added U? (x2): 74AHC138, symbol 74xx:74HC138
- added U?: 74AHC245, symbol AES_Library:74HC245-AES
- U?: value 74AHC541-AES -> 74AHC541
Connections:
- net BA3 is gone; now on net ZA3: U?.1 (A0)
- net BA4 is gone; now on net ZA4: U?.2 (A1)
- net BA5 is gone; now on net ZA5: U?.3 (A2)
- net +5V: now also U?.14 (VCC), U?.14 (VCC), U?.16 (VCC), U?.16 (VCC), U?.20 (VCC), U?.20 (VCC), U?.20 (VCC), U?.20 (VCC), U?.5 (VDD)
- net BA00: now also U?.18 (B0)
- net BA01: now also U?.17 (B1)
- net BA02: now also U?.16 (B2)
- net BA03: now also U?.15 (B3)
- net BA04: now also U?.14 (B4)
- net BA05: now also U?.13 (B5)
- net BA06: now also U?.12 (B6)
- net BA07: now also U?.11 (B7)
- net BA08: now also U?.18 (B0)
- net BA09: now also U?.17 (B1)
- net BA10: now also U?.16 (B2)
- net BA11: now also U?.15 (B3)
- net BA12: now also U?.14 (B4)
- net BA13: now also U?.11 (B0), U?.11 (B0)
- net BA14: now also U?.10 (B1), U?.10 (B1)
- net BA15: now also U?.9 (B2), U?.9 (B2)
- net BA16: now also U?.18 (B0)
- net BA17: now also U?.17 (B1)
- net BA18: now also U?.16 (B2)
- net BA19: now also U?.15 (B3)
- net BA20: now also U?.14 (B4)
- net BA21: now also U?.13 (B5)
- net BA22: now also U?.12 (B6)
- net BA23: now also U?.11 (B7)
- net BD0: now also U?.18 (B0)
- net BD1: now also U?.17 (B1)
- net BD2: now also U?.16 (B2)
- net BD3: now also U?.15 (B3)
- net BD4: now also U?.14 (B4)
- net BD5: now also U?.13 (B5)
- net BD6: now also U?.12 (B6)
- net BD7: now also U?.11 (B7)
- net BIORQ-: now also U?.3
- net BMREQ-: now also U?.3
- net GND: now also SW?.1, SW?.2, U?.10 (GND), U?.10 (GND), U?.10 (GND), U?.10 (GND), U?.19 (~{OE}), U?.19 (~{OE}), U?.19 (~{OE}), U?.2 (GND), U?.7 (GND), U?.7 (GND), U?.8 (GND), U?.8 (GND)
- net MEM_OP-: now also U?.22 (CE#), U?.22 (CE#), U?.1, U?.11, U?.12, U?.4 (~{E0}), U?.4 (~{E0})
- net NMI-: now also U?.8
- net NMIEN: now also U?.1
- net NOPAGE: now also U?.10, U?.6 (E2)
- net PA20: now also U?.13
- net PGINGEN: now also U?.11, U?.6 (E2)
- net RA55RO: now also U?.3 (A2)
- net RAMRD-: now also U?.6
- net RAMRDP-: now also U?.10 (~{Y5}), U?.5
- net RAMRDZ-: now also U?.10 (~{Y5}), U?.4
- net RAMWR-: now also U?.6
- net RAMWRP-: now also U?.5, U?.9 (~{Y6})
- net RAMWRZ-: now also U?.4, U?.9 (~{Y6})
- net ROMRD-: now also U?.6
- net ROMRDP-: now also U?.14 (~{Y1}), U?.5
- net ROMRDZ-: now also U?.14 (~{Y1}), U?.4
- net ROMWR-: now also U?.6
- net ROMWRP-: now also U?.13 (~{Y2}), U?.5
- net ROMWRZ-: now also U?.13 (~{Y2}), U?.4
- net ZA0: now also U?.2 (A0)
- net ZA1: now also U?.3 (A1)
- net ZA10: now also U?.4 (A2)
- net ZA11: now also U?.5 (A3)
- net ZA12: now also U?.6 (A4)
- net ZA13: now also U?.3 (A0)
- net ZA14: now also U?.4 (A1)
- net ZA15: now also U?.5 (A2)
- net ZA2: now also U?.2, U?.4 (A2)
- net ZA3: now also U?.5 (A3)
- net ZA4: now also U?.6 (A4)
- net ZA5: now also U?.7 (A5)
- net ZA6: now also U?.3, U?.8 (A6)
- net ZA7: now also U?.1, U?.9 (A7)
- net ZA8: now also U?.2 (A0)
- net ZA9: now also U?.3 (A1)
- net ZBSAK-: now also U?.1; no longer U?.1 (~{OEa}), U?.13 (OEb)
- net ZD0: now also U?.2 (A0)
- net ZD1: now also U?.3 (A1)
- net ZD2: now also U?.4 (A2)
- net ZD3: now also U?.5 (A3)
- net ZD4: now also U?.6 (A4)
- net ZD5: now also U?.7 (A5)
- net ZD6: now also U?.8 (A6)
- net ZD7: now also U?.9 (A7)
- net ZDIN-: now also U?.2, U?.2 (A1), U?.2 (A1), U?.5
- net ZDTOBD: now also U?.3; no longer U?.1 (A>B)
- net ZIORQ: no longer U?.22 (CE#), U?.22 (CE#)
- net ZIORQ-: now also U?.1, U?.4, U?.5
- net ZM1-: now also U?.2, U?.6
- net ZMASTER: now also U?.1 (~{OEa}), U?.13 (OEb), U?.1, U?.1 (A>B), U?.1 (A>B), U?.1 (A>B), U?.19 (~{OE}), U?.2, U?.2, U?.2, U?.2
- net ZNMI-: now also U?.9
- net ZRD-: now also U?.13, U?.13
- net ZRFSH-: now also U?.2
- net ZRST: now also U?.4
- net ZRST-: now also U?.2, U?.3
- net ZWR-: now also U?.1 (A0), U?.1 (A0)
- net BRDRST-: now reaches U?.1
- net BRDRST-: now also U?.1 (~{RST})
- net MHA21: now reaches RN?.7 (R6)
- net MHA21: now also U?.3, U?.7 (A5)
- net MHA22: now reaches RN?.8 (R7)
- net MHA22: now also U?.4, U?.8 (A6)
- net MHA23: now reaches RN?.9 (R8)
- net MHA23: now also U?.5, U?.9 (A7)
- net at U?.6 (E2): now also U?.3, U?.5
- net ZMASTER-: now reaches U?.19 (~{OE})
- net ZMASTER-: now also U?.3
- net BDRST- renamed BRSTREQ-
- net BRSTREQ-: now also SW?.3, SW?.4, U?.4 (~{MR})
- net LMA13 renamed MHA13
- net MHA13: now also U?.3 (A0)
- net LMA14 renamed MHA14
- net MHA14: now also U?.4 (A1)
- net LMA15 renamed MHA15
- net MHA15: now also U?.5 (A2)
- net LMA16 renamed MHA16
- net MHA16: now also U?.2 (A0)
- net LMA17 renamed MHA17
- net MHA17: now also U?.3 (A1)
- net LMA18 renamed MHA18
- net MHA18: now also U?.4 (A2)
- net LMA19 renamed MHA19
- net MHA19: now also U?.3 (A2), U?.5 (A3)
- net LMA20 renamed MHA20
- net MHA20: now also U?.2, U?.6 (A4)
- net LOCALI- renamed LCLIO-
- net LCLIO-: now also U?.1, U?.1, U?.4
- net ZPGPRS- renamed ZPGPRS
- new net: U?.1 (~{OEa}), U?.3 (x2)
- new net: U?.1, U?.13 (OEb) (x2)
- new net: U?.1, U?.5
- new net: U?.13, U?.3, U?.6
- new net: U?.2, U?.6
- new net: U?.10, U?.2
- new net BDZD-: U?.6
- new net BIACK-: U?.3, U?.5
- new net BUSRD-: U?.11, U?.4
- new net INTACK: U?.1, U?.1, U?.12, U?.4, U?.5
- new net LCLIEO: U?.2, U?.5
- new net LCLMEM-: U?.11, U?.2, U?.5
- new net LCLOP: U?.12, U?.3, U?.5
- new net LCLOP-: U?.12, U?.4, U?.6, U?.6
- new net LCLRD-: U?.1, U?.11
- new net LIACK-: U?.2, U?.3
- new net LOW1MEG-: U?.5 (~{E1}), U?.5 (~{E1}), U?.6
- new net MEM_OP: U?.1, U?.4
- new net ZBDEN-: U?.6
- new net ZD=>BD: U?.3
Other:
- moved on the sheet: OPT?, RN?, U?, U?A, U?B

Commit message: DBG: PR1.0, ZMB PR7.5, Timing diagrams
Parts:
- removed U? (x3): 74HC04, symbol AES_Library:7404-AES
- removed U? (x8): 74AHC08, symbol 74xx:74LS08
- removed U? (x9): 74HCT00, symbol 74xx:74HC00
- removed U? (x6): 74HCT32, symbol 74xx:74LS32
- removed U?: 74HC4002, symbol 4xxx:4002
- removed U? (x2): 74HCT86, symbol 74xx:74LS86
- removed U? (x2): 74HC02, symbol 74xx:74HC02
- removed U? (x2): 74HCT02, symbol 74xx:74HC02
- removed U?: 74AHC245, symbol AES_Library:74HC245-AES
- added U?: 74HCT00, symbol 74xx:74HC00
- added U?: 74HC4002, symbol 4xxx:4002
- added U?: 74HC04, symbol AES_Library:7404-AES
- added U?: 74AHC08, symbol 74xx:74LS08
- RN? (x3): value 20k -> 10k
Connections:
- net +5V: now also RN?.1 (common), RN?.1 (common), RN?.1 (common)
- net GND: no longer RN?.1 (common), RN?.1 (common), RN?.1 (common)
- net LOW1MEG-: now also U?.6
- net MEM_OP-: now also U?.3
- net MHA20: now also U?.2
- net MHA21: now also U?.3
- net MHA22: now also U?.4
- net MHA23: now also U?.5
- net ZBSAK-: now also U?.4
- net ZIORQ-: now also U?.1
- net ZMASTER: now also U?.6; no longer U?.1 (A>B), U?.1 (A>B), U?.1 (A>B)
- net ZRFSH-: now also U?.2
- net ZRST-: now also U?.5
- net ZMASTER-: no longer names the net of U?.19 (~{OE})
- new net: U?.1, U?.5
- new net ?ZA<=>BA?: U?.1 (A>B), U?.1 (A>B), U?.1 (A>B)
Other:
- moved on the sheet: OPT?, RN?, U?, U?A, U?B, U?E
