File: hw/SD-ZMB/History/PR7/logic_pwr_spr.kicad_sch (KiCad schematic)
At the start: 83 parts

Commit message: DBG: PR1.0, ZMB PR7.5, Timing diagrams
Parts:
- removed U? (x6): 74HCT32, symbol 74xx:74LS32
- removed U? (x9): 74HCT00, symbol 74xx:74HC00
- removed U? (x7): 74AHC08, symbol 74xx:74LS08
- removed U? (x2): 74HC02, symbol 74xx:74HC02
- removed U? (x2): 74HCT86, symbol 74xx:74LS86
- removed U? (x2): 74HCT02, symbol 74xx:74HC02
- removed U? (x2): 74HC04, symbol AES_Library:7404-AES
- added U (x2): 74ACT244, symbol 74xx:74AHCT244
Connections:
- net +5V: now also U.10 (GND), U.20 (VCC)
- net GND: now also U.10 (GND), U.20 (VCC)
- new net: U.1 (1OE), U.1 (1OE), U.19 (2OE), U.19 (2OE)
- new net BA0: U.18 (1Y0)
- new net BA1: U.16 (1Y1)
- new net BA10: U.14 (1Y2)
- new net BA11: U.12 (1Y3)
- new net BA12: U.3 (2Y0)
- new net BA13: U.5 (2Y1)
- new net BA14: U.7 (2Y2)
- new net BA15: U.9 (2Y3)
- new net BA2: U.14 (1Y2)
- new net BA3: U.12 (1Y3)
- new net BA4: U.3 (2Y0)
- new net BA5: U.5 (2Y1)
- new net BA6: U.7 (2Y2)
- new net BA7: U.9 (2Y3)
- new net BA8: U.18 (1Y0)
- new net BA9: U.16 (1Y1)
- new net ZA0: U.2 (1A0)
- new net ZA1: U.4 (1A1)
- new net ZA10: U.6 (1A2)
- new net ZA11: U.8 (1A3)
- new net ZA12: U.17 (2A0)
- new net ZA13: U.15 (2A1)
- new net ZA14: U.13 (2A2)
- new net ZA15: U.11 (2A3)
- new net ZA2: U.6 (1A2)
- new net ZA3: U.8 (1A3)
- new net ZA4: U.17 (2A0)
- new net ZA5: U.15 (2A1)
- new net ZA6: U.13 (2A2)
- new net ZA7: U.11 (2A3)
- new net ZA8: U.2 (1A0)
- new net ZA9: U.4 (1A1)
Other:
- moved on the sheet: J?, SW?, U?B, U?C, U?D, U?E, U?G
