File: hw/SD-DADPT/SD-DADPT.kicad_sch (KiCad schematic)
At the start: 16 parts, among them J1 CONN 1x8 Socket, J15 DISPLAY, J2 CONN 1x8 Socket, J3 CONN 1x6 Socket, J4 CONN 1x6 Socket, J5 CONN 1x22 SOCKET, J6 HDR 2x10 Pin, J7 CONN 1x6 HDR, J8 Screw_Terminal_01x02

Commit message: ZMB: v1.0 Board RFP
Parts:
- added H5: MountingHole, MountingHole:MountingHole_3.2mm_M3, symbol Mechanical:MountingHole
- J1: P3 (none) -> SPI_CLK; P4 (none) -> SPI_MISO; P5 (none) -> SPI_MOSI; P6 (none) -> SPI_SEL-; P7 (none) -> D1; P8 (none) -> D0
- J2: P1 (none) -> D7; P2 (none) -> D6; P3 (none) -> D5; P4 (none) -> D4; P5 (none) -> D3; P6 (none) -> D2
- J3: P1 (none) -> RD-; P2 (none) -> WR-; P3 (none) -> RS:C/D-; P4 (none) -> DSEL-; P5 (none) -> RST-
- J4: P2 (none) -> 3.3V; P3 (none) -> 5V; P5 (none) -> GND
- J5: P1 (none) -> FG; P10 (none) -> D0; P11 (none) -> D1; P12 (none) -> D2; P13 (none) -> D3; P14 (none) -> D4; P15 (none) -> D5; P16 (none) -> D6; P17 (none) -> D7; P18 (none) -> FS:F1/F0-; P19 (none) -> VEE(CONTV); P2 (none) -> VSS/GND; P20 (none) -> BL-A; P21 (none) -> BL-K; P22 (none) -> NC; P3 (none) -> VDD/5V; P4 (none) -> CONT/V0; P5 (none) -> WR-; P6 (none) -> RD-; P7 (none) -> DSEL-; P8 (none) -> RS:C/D-; P9 (none) -> RST-
- J6: FB (none) -> DISPLAY CABLE
- J7: P1 (none) -> GND; P2 (none) -> 5V; P3 (none) -> CLK; P4 (none) -> MISO; P5 (none) -> MOSI; P6 (none) -> SEL-
Connections:
- net D0: now also J1.8 (Pin_8); no longer J1.1 (Pin_1)
- net D1: now also J1.7 (Pin_7); no longer J1.2 (Pin_2)
- net SPI_CLK: now also J1.3 (Pin_3); no longer J1.6 (Pin_6)
- net SPI_MISO: now also J1.4 (Pin_4); no longer J1.5 (Pin_5)
- net SPI_MOSI: now also J1.5 (Pin_5); no longer J1.4 (Pin_4)
- net SPI_SEL-: now also J1.6 (Pin_6); no longer J1.3 (Pin_3)
Other:
- moved on the sheet: C2, J2, J3, J4, J7
