File: hw/SD-DBG/SD-DBG.kicad_sch (KiCad schematic)
At the start: 121 parts, among them J1 HDR 02x40 Pin (80)

Commit message: DBG: PR1.0, ZMB PR7.5, Timing diagrams
Parts:
- removed R?: 10k, symbol Device:R_Small_US
- removed SW?: SW Push Tactile, symbol AES_Library:SW_Push_Tactile_12-34
- removed U? (x3): 7404, symbol AES_Library:7404-AES
- removed U? (x3): 74HC08, symbol 74xx:74LS08
- removed U?: 74HC93, symbol AES_Library:7493-AES
- removed U?: 74HC05, symbol AES_Library:7405-AES
- removed U?: 74HC00, symbol 74xx:74LS00
- added C?: 50u, symbol Device:C_Polarized_US
- added J?: JACK BARREL DC, symbol AES_Library:BARREL_JACK-AES
- added J? (x2): HDR 2x9 Pins, symbol Connector_Generic:Conn_02x09_Row_Letter_First
- added R?: 10k, symbol Device:R_Small_US
- added SW?: SW Push Tactile, symbol AES_Library:SW_Push_Tactile_12-34
- added U? (x3): 74HC08, symbol 74xx:74LS08
- added U? (x2): 74HC164, symbol 74xx:74HC164
- added U? (x3): 74LS688, symbol 74xx:74LS688
- added U?: 74HC05, symbol AES_Library:7405-AES
- added U? (x3): 74HCT273, symbol 74xx:74HCT273
- added U? (x4): 74HC04, symbol AES_Library:7404-AES
- added U? (x3): 74HC74, symbol 74xx:74LS74
- added U?: 74HC138, symbol 74xx:74HC138
- added U?: 7404, symbol AES_Library:7404-AES
- added U?: 74HC00, symbol 74xx:74LS00
Connections:
- net +5V: now also U?.14 (VCC), U?.14 (VCC), U?.14 (VCC), U?.14 (VCC), U?.14 (VCC), R?.2, U?.14 (VCC), U?.16 (VCC), U?.20 (VCC), U?.20 (VCC), U?.20 (VCC), U?.20 (VCC), U?.20 (VCC)
- net +5VL: now also C?.1, J?.1
- net A00: now also U?.1 (A0), U?.17 (P7)
- net A01: now also U?.15 (P6), U?.2 (A1)
- net A02: now also U?.9, U?.13 (P5)
- net A03: now also U?.10, U?.11 (P4)
- net A04: now also U?.13, U?.8 (P3)
- net A05: now also U?.2, U?.6 (P2)
- net A06: now also U?.13, U?.4 (P1)
- net A07: now also U?.11, U?.2 (P0)
- net A08: now also U?.17 (P7)
- net A09: now also U?.15 (P6)
- net A10: now also U?.13 (P5)
- net A11: now also U?.11 (P4)
- net A12: now also U?.8 (P3)
- net A13: now also U?.6 (P2)
- net A14: now also U?.4 (P1)
- net A15: now also U?.2 (P0)
- net A16: now also U?.17 (P7)
- net A17: now also U?.15 (P6)
- net A18: now also U?.13 (P5)
- net A19: now also U?.11 (P4)
- net A20: now also U?.8 (P3)
- net A21: now also U?.6 (P2)
- net A22: now also U?.4 (P1)
- net A23: now also U?.2 (P0)
- net BRDRST-: now also U?.1 (~{Mr}), U?.1 (~{Mr}), U?.1 (~{Mr}), U?.1 (~{R})
- net CLK: now also U?.8 (CP), U?.8 (CP)
- net D0: now also U?.2 (D), U?.3 (D0), U?.3 (D0), U?.3 (D0)
- net D1: now also U?.4 (D1), U?.4 (D1), U?.4 (D1)
- net D2: now also U?.7 (D2), U?.7 (D2), U?.7 (D2)
- net D3: now also U?.8 (D3), U?.8 (D3), U?.8 (D3)
- net D4: now also U?.13 (D4), U?.13 (D4), U?.13 (D4)
- net D5: now also U?.14 (D5), U?.14 (D5), U?.14 (D5)
- net D6: now also U?.17 (D6), U?.17 (D6), U?.17 (D6)
- net D7: now also U?.18 (D7), U?.18 (D7), U?.18 (D7)
- net GND: now also U?.1 (~{G1}), U?.1 (~{G1}), U?.1 (~{G1}), U?.1 (~{G1}), U?.1 (~{G1}), U?.19 (~{G2}), U?.19 (~{G2}), U?.19 (~{G2}), U?.19 (~{G2}), U?.19 (~{G2}), U?.7 (GND), U?.7 (GND), U?.7 (GND), U?.7 (GND), U?.7 (GND), C?.2, J?.2, SW?.1, SW?.2, U?.1 (G), U?.10 (GND), U?.10 (GND), U?.10 (GND), U?.10 (GND), U?.10 (GND), U?.10 (GND), U?.7 (GND), U?.8 (GND)
- net IF-: now also U?.11 (C)
- net IORQ-: now also U?.5
- net M1: now also U?.10
- net MREQ-: now also U?.5
- net PU?: now also J?.a1 (Pin_a1), J?.a1 (Pin_a1), U?.1 (DSA), U?.1 (DSA), U?.13 (~{R}), U?.2 (DSB), U?.2 (DSB), U?.4 (~{S})
- net WAIT-: now also U?.8, U?.6
- net WR-: now also U?.5 (~{E1})
- net ZSR-: now also U?.6
- net IOWAIT: now reaches U?.9
- net IOWAIT: now also J?.b1 (Pin_b1), J?.b2 (Pin_b2), J?.b3 (Pin_b3), J?.b4 (Pin_b4), J?.b5 (Pin_b5), J?.b6 (Pin_b6), J?.b7 (Pin_b7), J?.b8 (Pin_b8), J?.b9 (Pin_b9)
- net IFABRK-: now reaches U?.4
- net IFABRK-: now also U?.9 (Q)
- net PBBRK-: now reaches U?.5
- net PBBRK-: now also R?.1, SW?.3, SW?.4
- net at U?.6: now also U?.9 (~{MR})
- net at U?.8: now also U?.3 (A2)
- new net: U?.13, U?.8
- new net: U?.1 (G), U?.19 (P=R) (x2)
- new net: U?.12 (Q4), U?.12 (R4) (x3)
- new net: U?.14 (R5), U?.15 (Q5) (x3)
- new net: U?.16 (Q6), U?.16 (R6) (x3)
- new net: U?.18 (R7), U?.19 (Q7) (x3)
- new net: U?.2 (Q0), U?.3 (R0) (x3)
- new net: U?.5 (Q1), U?.5 (R1) (x3)
- new net: U?.6 (Q2), U?.7 (R2) (x3)
- new net: U?.9 (Q3), U?.9 (R3) (x3)
- new net: U?.1, U?.12
- new net: U?.12, U?.3
- new net: U?.11, U?.4 (~{E0})
- new net: U?.11, U?.6 (E2)
- new net: U?.10, U?.12
- new net ADDREQ-: U?.12 (D), U?.19 (P=R)
- new net BRKADRH-: U?.11 (Cp), U?.13 (~{Y2})
- new net BRKADRL-: U?.11 (Cp), U?.15 (~{Y0})
- new net BRKADRM-: U?.11 (Cp), U?.14 (~{Y1})
- new net BRKDABL-: U?.10 (~{S}), U?.5 (Q)
- new net BRKENWR-: U?.12 (~{Y3}), U?.3 (C)
- new net IORQ: U?.6, U?.9, U?.9 (~{MR})
- new net IOWAIT1: J?.a2 (Pin_a2), U?.3 (Q0)
- new net IOWAIT2: J?.a3 (Pin_a3), U?.4 (Q1)
- new net IOWAIT3: J?.a4 (Pin_a4), U?.5 (Q2)
- new net IOWAIT4: J?.a5 (Pin_a5), U?.6 (Q3)
- new net IOWAIT5: J?.a6 (Pin_a6), U?.10 (Q4)
- new net IOWAIT6: J?.a7 (Pin_a7), U?.11 (Q5)
- new net IOWAIT7: J?.a8 (Pin_a8), U?.12 (Q6)
- new net IOWAIT8: J?.a9 (Pin_a9), U?.13 (Q7)
- new net MWAIT: J?.b1 (Pin_b1), J?.b2 (Pin_b2), J?.b3 (Pin_b3), J?.b4 (Pin_b4), J?.b5 (Pin_b5), J?.b6 (Pin_b6), J?.b7 (Pin_b7), J?.b8 (Pin_b8), J?.b9 (Pin_b9), U?.5
- new net MWAIT1: J?.a2 (Pin_a2), U?.3 (Q0)
- new net MWAIT2: J?.a3 (Pin_a3), U?.4 (Q1)
- new net MWAIT3: J?.a4 (Pin_a4), U?.5 (Q2)
- new net MWAIT4: J?.a5 (Pin_a5), U?.6 (Q3)
- new net MWAIT5: J?.a6 (Pin_a6), U?.10 (Q4)
- new net MWAIT6: J?.a7 (Pin_a7), U?.11 (Q5)
- new net MWAIT7: J?.a8 (Pin_a8), U?.12 (Q6)
- new net MWAIT8: J?.a9 (Pin_a9), U?.13 (Q7)
Other:
- moved on the sheet: J1, R?, SW?, U?A, U?B, U?C, U?D, U?E, U?F, U?G

Commit message: ZMB: Diagrams and start of PCB. DBG: Updated WAIT. DADPT: Display/Cable PCB ordered.
Parts:
- removed C?: 50u, symbol Device:C_Polarized_US
- removed D? (x40): LED RED, symbol Device:LED
- removed J?: JACK BARREL DC, symbol AES_Library:BARREL_JACK-AES
- removed J? (x2): HDR 2x9 Pins, symbol Connector_Generic:Conn_02x09_Row_Letter_First
- removed R? (x40): 510, symbol Device:R_Small_US
- removed U? (x5): 74HC04, symbol AES_Library:7404-AES
- removed U? (x4): 74HC08, symbol 74xx:74LS08
- removed U?: 74HCT541, symbol AES_Library:74541-AES
- removed U? (x4): 74HC74, symbol 74xx:74LS74
- removed U? (x2): 74HC164, symbol 74xx:74HC164
- removed U? (x5): 74HC05, symbol AES_Library:7405-AES
- removed U? (x3): 74LS688, symbol 74xx:74LS688
- removed U? (x5): 74HC00, symbol 74xx:74LS00
- removed U? (x4): 74HCT540, symbol AES_Library:74540-AES
- removed U? (x2): 7404, symbol AES_Library:7404-AES
- added D? (x8): LED RED, symbol Device:LED
- added J? (x2): HDR 2x9 Pins, symbol Connector_Generic:Conn_02x09_Row_Letter_First
- added Opt?: HDR 1x3 Pin, symbol AES_Library:AES-Opt_1_of_2
- added R? (x8): 510, symbol Device:R_Small_US
- added U? (x3): 74AHCT00, symbol 74xx:74LS00
- added U? (x3): 74AHCT04, symbol AES_Library:7404-AES
- added U? (x2): 74AHCT10, Package_SO:SOIC-14_3.9x8.7mm_P1.27mm, symbol 74xx:74LS10
- added U? (x4): 74F260, symbol AES_Library:74F260-AES
- added U? (x6): 74F27, symbol 74xx:74LS27
- added U? (x4): 74HCT574, symbol AES_Library:74574-AES
- added U? (x10): 74AHCT32, symbol 74xx:74LS32
- added U? (x5): 74AHCT02, symbol 74xx:74LS02
- added U? (x2): 74HC164, symbol 74xx:74HC164
- added U?: 74AHCT273, symbol AES_Library:74273-AES
- added U? (x2): 74F27, Package_SO:SOIC-14_3.9x8.7mm_P1.27mm, symbol 74xx:74LS27
- added U? (x4): 74AHCT74, symbol 74xx:74LS74
- added U? (x3): 74HCT688, symbol AES_Library:74688-AES
- added U?: 74ACT138, symbol 74xx:74HC138
- added U?: 74AHC541, Package_SO:SOIC-20W_7.5x12.8mm_P1.27mm, symbol AES_Library:74AHC541-AES
- added U? (x2): 74AHC05, symbol AES_Library:7405-AES
- added U?: 74HCT161, symbol AES_Library:74161-AES
- U? (x2): value 74HC74 -> 74AHCT74
- U? (x2): value 74HC04 -> 74AHCT04
- U? (x3): value 74HCT273 -> 74AHCT273
- U?: value 74HC08 -> 74AHCT08
- U?: value 74HC00 -> 74AHCT00
- U? (x2): value 74HC05 -> 74AHC05
- U?: value 74HC138 -> 74ACT138
- U?: value 7404 -> 74AHCT04
Connections:
- net +5V: now also U?.20 (VCC), R?.2, R?.2, R?.2, R?.2, R?.2, R?.2, R?.2, R?.2, U?.14 (VCC), U?.14 (VCC), U?.16 (VCC), U?.16 (VCC), U?.20 (VCC), U?.20 (VCC), U?.20 (VCC), U?.20 (VCC), U?.20 (VCC), U?.20 (VCC), U?.20 (VCC), U?.20 (VCC), U?.20 (VCC)
- net A00: now also U?.17 (P7), U?.9 (D7)
- net A01: now also U?.15 (P6), U?.8 (D6)
- net A02: now also U?.3 (A2), U?.13 (P5), U?.7 (D5)
- net A03: now also U?.4 (~{E0}), U?.11 (P4), U?.6 (D4)
- net A04: now also U?.1, U?.5 (D3), U?.8 (P3)
- net A05: now also U?.12, U?.4 (D2), U?.6 (P2)
- net A06: now also U?.13, U?.3 (D1), U?.4 (P1)
- net A07: now also U?.2, U?.2 (D0), U?.2 (P0)
- net A08: now also U?.17 (P7), U?.9 (D7)
- net A09: now also U?.15 (P6), U?.8 (D6)
- net A10: now also U?.13 (P5), U?.7 (D5)
- net A11: now also U?.11 (P4), U?.6 (D4)
- net A12: now also U?.5 (D3), U?.8 (P3)
- net A13: now also U?.4 (D2), U?.6 (P2)
- net A14: now also U?.3 (D1), U?.4 (P1)
- net A15: now also U?.2 (D0), U?.2 (P0)
- net A16: now also U?.17 (P7), U?.9 (D7)
- net A17: now also U?.15 (P6), U?.8 (D6)
- net A18: now also U?.13 (P5), U?.7 (D5)
- net A19: now also U?.11 (P4), U?.6 (D4)
- net A20: now also U?.5 (D3), U?.8 (P3)
- net A21: now also U?.4 (D2), U?.6 (P2)
- net A22: now also U?.3 (D1), U?.4 (P1)
- net A23: now also U?.2 (D0), U?.2 (P0)
- net BRDRST-: now also U?.1 (~{Mr}), U?.13 (~{R})
- net CLK: now also U?.11 (C), U?.8 (CP), U?.8 (CP)
- net D0: now also U?.19 (Q0), U?.19 (Q0), U?.19 (Q0), U?.19 (Q0)
- net D1: now also U?.18 (Q1), U?.18 (Q1), U?.18 (Q1), U?.18 (Q1)
- net D2: now also U?.17 (Q2), U?.17 (Q2), U?.17 (Q2), U?.17 (Q2)
- net D3: now also U?.16 (Q3), U?.16 (Q3), U?.16 (Q3), U?.16 (Q3)
- net D4: now also U?.15 (Q4), U?.15 (Q4), U?.15 (Q4), U?.15 (Q4)
- net D5: now also U?.14 (Q5), U?.14 (Q5), U?.14 (Q5), U?.14 (Q5)
- net D6: now also U?.13 (Q6), U?.13 (Q6), U?.13 (Q6), U?.13 (Q6)
- net D7: now also U?.12 (Q7), U?.12 (Q7), U?.12 (Q7), U?.12 (Q7)
- net GND: now also Opt?.1 (Pin_A), U?.1 (~{EIN}), U?.1 (~{EIN}), U?.1 (~{EIN}), U?.1 (~{G1}), U?.10 (GND), U?.10 (GND), U?.10 (GND), U?.10 (GND), U?.10 (GND), U?.10 (GND), U?.10 (GND), U?.10 (GND), U?.10 (GND), U?.12 (D), U?.13, U?.13, U?.13, U?.19 (~{G2}), U?.3 (A2), U?.3 (D0), U?.4, U?.4 (D1), U?.4 (~{E0}), U?.5, U?.5 (D2), U?.5 (~{E1}), U?.6 (D3), U?.7 (GND), U?.7 (GND), U?.8 (GND), U?.8 (GND)
- net HALT-: now also U?.7 (A5)
- net IF-: now also U?.12, U?.3 (C), U?.9
- net INT-: now also U?.8 (A6)
- net IORQ: now also U?.6, U?.9 (~{MR})
- net IORQ-: now also U?.13, U?.2, U?.2, U?.2, U?.3, U?.3 (A1), U?.5
- net IOWAIT1: now also J?.a2 (Pin_a2), U?.3 (Q0)
- net IOWAIT2: now also J?.a3 (Pin_a3), U?.4 (Q1)
- net IOWAIT3: now also J?.a4 (Pin_a4), U?.5 (Q2)
- net IOWAIT4: now also J?.a5 (Pin_a5), U?.6 (Q3)
- net IOWAIT5: now also J?.a6 (Pin_a6), U?.10 (Q4)
- net IOWAIT6: now also J?.a7 (Pin_a7), U?.11 (Q5)
- net IOWAIT7: now also J?.a8 (Pin_a8), U?.12 (Q6)
- net IOWAIT8: now also J?.a9 (Pin_a9), U?.13 (Q7)
- net M1: now also U?.1, U?.12, U?.2, U?.9
- net MREQ-: now also U?.2, U?.2, U?.2, U?.2 (A0), U?.3
- net MWAIT1: now also J?.a2 (Pin_a2), U?.3 (Q0)
- net MWAIT2: now also J?.a3 (Pin_a3), U?.4 (Q1)
- net MWAIT3: now also J?.a4 (Pin_a4), U?.5 (Q2)
- net MWAIT4: now also J?.a5 (Pin_a5), U?.6 (Q3)
- net MWAIT5: now also J?.a6 (Pin_a6), U?.10 (Q4)
- net MWAIT6: now also J?.a7 (Pin_a7), U?.11 (Q5)
- net MWAIT7: now also J?.a8 (Pin_a8), U?.12 (Q6)
- net MWAIT8: now also J?.a9 (Pin_a9), U?.13 (Q7)
- net NMI-: now also U?.9 (A7)
- net PBBRK-: now also U?.9 (D7)
- net PBCRST-: now also U?.5
- net PU?: now also J?.a1 (Pin_a1), J?.a1 (Pin_a1), U?.1 (DSA), U?.1 (DSA), U?.10 (CET), U?.10 (~{S}), U?.2 (D), U?.2 (DSB), U?.2 (DSB), U?.4 (~{S}), U?.4 (~{S}), U?.6 (E2), U?.9 (~{PE})
- net RD-: now also U?.10, U?.10, U?.10, U?.10, U?.13, U?.13, U?.5 (A3)
- net WAIT-: now also U?.6, U?.6 (A4), U?.8
- net WR-: now also U?.10, U?.10, U?.10, U?.13, U?.13, U?.4 (A2), U?.9; no longer U?.5 (~{E1})
- net at U?.12 (Q4): now also U?.12 (R4) (x3)
- net at U?.15 (Q5): now also U?.14 (R5) (x3)
- net at U?.16 (Q6): now also U?.16 (R6) (x3)
- net at U?.19 (Q7): now also U?.18 (R7) (x3)
- net at U?.2 (Q0): now also U?.3 (R0) (x3)
- net at U?.5 (Q1): now also U?.5 (R1) (x3)
- net at U?.6 (Q2): now also U?.7 (R2) (x3)
- net at U?.9 (Q3): now also U?.9 (R3) (x3)
- net SPCRST-: now reaches U?.3
- net SPCRST-: now also U?.10 (~{S}), U?.4
- net IO_65-: now reaches U?.10 (~{Y5})
- net IO_64-: now reaches U?.11 (~{Y4})
- net at U?.6 (E2): now also U?.5
- net IO_67-: now reaches U?.7 (~{Y7})
- net IO_66-: now reaches U?.9 (~{Y6})
- net at U?.1: now also U?.6
- net BRKADRH-: no longer names the net of U?.11 (Cp)
- net BRKADRH-: now also U?.8; no longer U?.13 (~{Y2})
- net BRKADRL-: no longer names the net of U?.11 (Cp)
- net BRKADRL-: now also U?.8; no longer U?.15 (~{Y0})
- net BRKADRM-: no longer names the net of U?.11 (Cp)
- net BRKADRM-: now also U?.8; no longer U?.14 (~{Y1})
- net BRKENWR- renamed BRKCTRL-
- net BRKCTRL-: now also U?.10, U?.9
- net IFABRK- renamed BRKCM-
- net BRKCM-: now also U?.2 (D0), U?.8
- new net: D?.1 (K), U?.12 (Y6)
- new net: D?.2 (A), R?.1 (x8)
- new net: D?.1 (K), U?.17 (Y1)
- new net: U?.10, U?.6
- new net: U?.13, U?.8
- new net: U?.12, U?.9
- new net: D?.1 (K), U?.16 (Y2)
- new net: D?.1 (K), U?.11 (Y7)
- new net: U?.1 (~{OE}), U?.8 (x4)
- new net: U?.1, U?.9
- new net: U?.3 (C), U?.8
- new net: U?.12 (D), U?.5 (Q)
- new net: U?.12, U?.7 (CEP)
- new net: U?.13, U?.6
- new net: Opt?.2 (Pin_Common), U?.2
- new net: U?.2 (D), U?.6 (~{Q})
- new net: U?.2 (CP), U?.5 (Q)
- new net: D?.1 (K), U?.13 (Y5)
- new net: U?.11, U?.5 (~{E1})
- new net: D?.1 (K), U?.15 (Y3)
- new net: U?.1, U?.9 (~{MR})
- new net: U?.1, U?.5
- new net: D?.1 (K), U?.14 (Y4)
- new net: D?.1 (K), U?.18 (Y0)
- new net ADR16CM: U?.12, U?.3
- new net ADR24CM: U?.2, U?.5
- new net ADR8CM: U?.1, U?.12
- new net ADRHEQ-: U?.19 (~{P=R}), U?.2
- new net ADRHSEL-: U?.13 (~{Y2}), U?.9, U?.9
- new net ADRLEQ-: U?.12, U?.13, U?.19 (~{P=R}), U?.3
- new net ADRLSEL-: U?.15 (~{Y0}), U?.9, U?.9
- new net ADRMEQ-: U?.19 (~{P=R}), U?.2, U?.3
- new net ADRMSEL-: U?.14 (~{Y1}), U?.9, U?.9
- new net BADRCM-: U?.5, U?.8 (D6), U?.9
- new net BCADRA: U?.1, U?.8
- new net BCMAD16-: U?.1, U?.13 (~{Y2})
- new net BCMAD24-: U?.1, U?.12 (~{Y3})
- new net BCMAD8-: U?.14 (~{Y1}), U?.2
- new net BCMADA-: U?.15 (~{Y0}), U?.9
- new net BDCTLWR-: U?.11 (Cp), U?.8
- new net BIFCM: U?.10, U?.11, U?.7 (D5)
- new net BIRCM: U?.12, U?.3 (D1), U?.4
- new net BIWCM: U?.12, U?.4 (D2), U?.8
- new net BMRCM: U?.12, U?.5 (D3), U?.9
- new net BMWCM: U?.10, U?.12, U?.6 (D4)
- new net BOPCM-: U?.10, U?.6
- new net BRKIF-: U?.16 (Q6), U?.8
- new net BRKIOR-: U?.1, U?.6 (Q2)
- new net BRKIOW-: U?.1, U?.9 (Q3)
- new net BRKMR-: U?.1, U?.12 (Q4)
- new net BRKMW-: U?.1, U?.15 (Q5)
- new net BRKOP0: U?.1 (A0), U?.2 (Q0)
- new net BRKOP1: U?.2 (A1), U?.5 (Q1)
- new net BUSMEM-: Opt?.3 (Pin_B), U?.12
- new net DBMODE-: U?.10, U?.8 (~{Q})
- new net IOWAITRQ-: J?.b1 (Pin_b1), J?.b2 (Pin_b2), J?.b3 (Pin_b3), J?.b4 (Pin_b4), J?.b5 (Pin_b5), J?.b6 (Pin_b6), J?.b7 (Pin_b7), J?.b8 (Pin_b8), J?.b9 (Pin_b9), U?.3
- new net MHA20: U?.1
- new net MHA21: U?.2
- new net MHA22: U?.13
- new net MHA23: U?.3
- new net MWAITRQ-: J?.b1 (Pin_b1), J?.b2 (Pin_b2), J?.b3 (Pin_b3), J?.b4 (Pin_b4), J?.b5 (Pin_b5), J?.b6 (Pin_b6), J?.b7 (Pin_b7), J?.b8 (Pin_b8), J?.b9 (Pin_b9), U?.3
- new net SAVEPC: U?.11 (Cp), U?.11 (Cp), U?.11 (Cp), U?.11 (Cp), U?.9 (Q)
- new net SWTOUM: U?.1 (~{MR}), U?.1 (~{R}), U?.19 (Q7), U?.5
- new net UMSWTCH: U?.1, U?.11 (C), U?.15 (TC), U?.2
- new net USRMODE-: U?.1 (~{R}), U?.13 (~{R}), U?.9 (Q)
- new net ZD0: U?.3 (D0)
- new net ZD1: U?.4 (D1)
- new net ZD2: U?.7 (D2)
- new net ZD3: U?.8 (D3)
- new net ZD4: U?.13 (D4)
- new net ZD5: U?.14 (D5)
- new net ZD6: U?.17 (D6)
- new net ZD7: U?.18 (D7)
- new net ZIORQ-: U?.1
- new net ZRFSH-: U?.2
Other:
- added sheet BlinkenLights & Pwr (blinkenlights.kicad_sch)
- note removed: "DER BLINKENLIGHTS"
- moved on the sheet: J1, SW?, U?, U?A, U?B

Commit message: ZMB: v1.0 w/Spares added. RFP
Connections:
- net CPURST-: now also J1.40 (~{CPURSTRQ}); no longer J1.60 (~{CPURST})
- net at J1.38 (IEI): now also J1.39 (IEO)
- net at J1.42 (BAI): now also J1.43 (BAO)
Other:
- moved on the sheet: D?, R?, U?, U?A, U?B, U?C

Commit message: PCB received
Parts:
- U?: value 74HCT688 -> 74FCT521; ALT (none) -> (74HCT688)
